File: LinkSocket.kicad_sch (KiCad schematic)
At the start: 4 parts, among them J201 NE8FAH, U201 THVD2442

Commit message: Update Library
Parts:
- C201: symbol V2_Device:C_0603_0u1 -> V2_Capacitor:0603_0u1
- R201: symbol V2_Device:R_0603_100R -> V2_Resistor:0603_100R
Changed lines of the file:
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@@
 		(on_board yes)
 		(dnp no)
-		(property "Reference" "#PWR0201"
+		(property "Reference" "#PWR201"
 			(at 154.94 62.23 0)
 			(effects
@@
 			(project "connect"
 				(path "/6c8448b4-b04d-47e1-934e-e40cbe27a7be/a64f4585-dd42-4120-8007-516d9ffa6e9b"
-					(reference "#PWR0201")
+					(reference "#PWR201")
 					(unit 1)
 				)
@@
 		(on_board yes)
 		(dnp no)
-		(property "Reference" "#PWR0203"
+		(property "Reference" "#PWR203"
 			(at 154.94 102.87 0)
 			(effects
@@
 			(project "connect"
 				(path "/6c8448b4-b04d-47e1-934e-e40cbe27a7be/a64f4585-dd42-4120-8007-516d9ffa6e9b"
-					(reference "#PWR0203")
+					(reference "#PWR203")
 					(unit 1)
 				)
@@
 		(on_board yes)
 		(dnp no)
-		(property "Reference" "#PWR0202"
+		(property "Reference" "#PWR202"
 			(at 176.53 69.85 0)
 			(effects
@@
 			(project "connect"
 				(path "/6c8448b4-b04d-47e1-934e-e40cbe27a7be/a64f4585-dd42-4120-8007-516d9ffa6e9b"
-					(reference "#PWR0202")
-					(unit 1)
-				)
-			)
-		)
-	)
-	(symbol
-		(lib_id "V2_Device:R_0603_100R")
+					(reference "#PWR202")
+					(unit 1)
+				)
+			)
+		)
+	)
+	(symbol
+		(lib_id "V2_Resistor:0603_100R")
 		(at 167.64 76.2 0)
 		(unit 1)
@@
 		(on_board yes)
 		(dnp no)
-		(property "Reference" "#PWR0204"
+		(property "Reference" "#PWR204"
 			(at 138.43 118.11 0)
 			(effects
@@
 			(project "connect"
 				(path "/6c8448b4-b04d-47e1-934e-e40cbe27a7be/a64f4585-dd42-4120-8007-516d9ffa6e9b"
-					(reference "#PWR0204")
-					(unit 1)
-				)
-			)
-		)
-	)
-	(symbol
-		(lib_id "V2_Device:C_0603_0u1")
+					(reference "#PWR204")
+					(unit 1)
+				)
+			)
+		)
+	)
+	(symbol
+		(lib_id "V2_Capacitor:0603_0u1")
 		(at 176.53 60.96 0)
 		(unit 1)
