File: LinkSocket.kicad_sch (KiCad schematic)
At the start: 4 parts, among them J201 NE8FAH, U201 THVD2442

Commit message: Refresh
Other:
- note added: "PoE Passive +28V IEEE 802.3af Mode B"
- note removed: "PoE Passive +24V IEEE 802.3af Mode B"
Changed lines of the file:
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@@
 		(company "Socket")
 	)
-	(text "PoE Passive +24V\nIEEE 802.3af Mode B"
+	(text "PoE Passive +28V\nIEEE 802.3af Mode B"
 		(exclude_from_sim no)
 		(at 169.164 150.876 0)

Commit message: KiCad 10
Other:
- company: Socket -> Versio Duo

Commit message: Refresh
Other:
- title: V2 Link -> V2 connect
Changed lines of the file:
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@@
 	(paper "A4")
 	(title_block
-		(title "V2 Link")
-		(date "2026-03-24")
+		(title "V2 connect")
+		(date "2026-03-26")
 		(rev "2026-03-14")
 		(company "Versio Duo")
