File: LinkSocket.kicad_sch (KiCad schematic)
At the start: 4 parts, among them J201 NE8FAH, U201 THVD2442

Commit message: Update
Parts:
- C201: Id (none) -> Capacitor:${SYMBOL_NAME}
- R201: Id (none) -> Resistor:${SYMBOL_NAME}
- U201: Id (none) -> RS485:${SYMBOL_NAME}
Changed lines of the file:
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@@
+			)
+		)
+		(property "Id" "RS485:${SYMBOL_NAME}"
+			(at 154.94 113.03 0)
+			(hide yes)
+			(show_name no)
+			(do_not_autoplace no)
+			(effects
+				(font
+					(size 1.27 1.27)
+				)
 			)
 		)
@@
 			)
 		)
+		(property "Id" "Resistor:${SYMBOL_NAME}"
+			(at 167.64 90.17 0)
+			(hide yes)
+			(show_name no)
+			(do_not_autoplace no)
+			(effects
+				(font
+					(size 1.27 1.27)
+				)
+			)
+		)
 		(pin "1"
 		)
@@
 			(hide yes)
 			(show_name no)
+			(do_not_autoplace no)
+			(effects
+				(font
+					(size 1.27 1.27)
+				)
+			)
+		)
+		(property "Id" "Capacitor:${SYMBOL_NAME}"
+			(at 176.53 76.2 0)
+			(hide yes)
+			(show_name no)

Commit message: Update
Parts:
- J201: Id (none) -> EtherCon:${SYMBOL_NAME}; Rating (none) -> CAT5e
- U201: Rating (none) -> 20Mbps
Changed lines of the file:
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@@
+			)
+		)
+		(property "Rating" "20Mbps"
+			(at 156.21 120.65 0)
+			(hide yes)
+			(show_name no)
+			(do_not_autoplace no)
+			(effects
+				(font
+					(size 1.27 1.27)
+				)
 			)
 		)
@@
 			(do_not_autoplace no)
 			(effects
+				(font
+					(size 1.27 1.27)
+				)
+			)
+		)
+		(property "Id" "EtherCon:${SYMBOL_NAME}"
+			(at 154.94 157.48 0)
+			(hide yes)
+			(show_name no)
+			(do_not_autoplace no)
+			(effects
+				(font
+					(size 1.27 1.27)
+				)
+			)
+		)
+		(property "Rating" "CAT5e"
+			(at 154.94 170.18 0)
+			(hide yes)
+			(show_name no)
+			(do_not_autoplace no)
+			(effects
