File: MIDIIn.kicad_sch (KiCad schematic)
At the start: 6 parts, among them J301 SJ2-25404B-SMT-TR, U301 TLP2361

Commit message: Update Library
Parts:
- C301, C302: symbol V2_Device:C_0603_0u1 -> V2_Capacitor:0603_0u1
- R301: symbol V2_Device:R_0603_220R -> V2_Resistor:0603_220R
