File: MIDIIn.kicad_sch (KiCad schematic)
At the start: 6 parts, among them J301 SJ2-25404B-SMT-TR, U301 TLP2361

Commit message: Replace diode
Parts:
- D301: value RB501SM -> PMEG2010EPK; footprint V2_Diode_SMD:D_SOD-523 -> V2_Diode_SMD:D_SOD-1608; symbol V2_Diode:RB501SM -> V2_Diode:PMEG2010EPK; Manufacturer ROHM Semiconductor -> Nexperia; Mouser 755-RB501SM-30FHT2R -> 771-PMEG2010EPK; Product RB501SM-30FHT2R -> PMEG2010EPK; Rating (none) -> 20V
Changed lines of the file:
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@@
 	(title_block
 		(title "MIDI In")
-		(date "2026-02-12")
-		(rev "2026-02-12")
+		(date "2026-03-12")
+		(rev "2026-03-12")
 	)

Commit message: KiCad 10
Other:
- company: (none) -> Versio Duo
Changed lines of the file:
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@@
 (kicad_sch
-	(version 20250114)
+	(version 20260306)
 	(generator "eeschema")
-	(generator_version "9.0")
+	(generator_version "10.0")
 	(paper "A4")
 	(title_block
 		(title "MIDI In")
-		(date "2026-03-12")
-		(rev "2026-03-12")
+		(date "2026-03-20")
+		(rev "2026-03-14")
+		(company "Versio Duo")
 	)

Commit message: Refresh
Other:
- title: MIDI In -> V2 connect
Changed lines of the file:
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@@
 	(paper "A4")
 	(title_block
-		(title "MIDI In")
-		(date "2026-03-24")
+		(title "V2 connect")
+		(date "2026-03-26")
 		(rev "2026-03-14")
 		(company "Versio Duo")
