File: MIDIIn.kicad_sch (KiCad schematic)
At the start: 6 parts, among them J301 SJ2-25404B-SMT-TR, U301 TLP2361

Commit message: Update
Parts:
- C301, C302: Id (none) -> Capacitor:${SYMBOL_NAME}
- D301: Id (none) -> Diode:${SYMBOL_NAME}
- J301: Id (none) -> Audio:${SYMBOL_NAME}
- R301: Id (none) -> Resistor:${SYMBOL_NAME}
- U301: Id (none) -> Optocoupler:${SYMBOL_NAME}

Commit message: Update
Parts:
- renumbered C302 to C301, C301 to C302
Changed lines of the file:
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@@
 		(rev "2026-03-28")
 		(company "Versio Duo")
+		(comment 1 "V2 Link Connector")
 	)

Commit message: Update
Parts:
- J301: Rating (none) -> 2.5mm
- U301: Rating (none) -> 15Mbps
Changed lines of the file:
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@@
 	(title_block
 		(title "V2 connect")
-		(date "2026-03-28")
-		(rev "2026-03-28")
+		(date "2026-04-14")
+		(rev "2026-04-14")
 		(company "Versio Duo")
 		(comment 1 "V2 Link Connector")
