File: MIDIOut.kicad_sch (KiCad schematic)
At the start: 6 parts, among them J401 SJ2-25404B-SMT-TR, U401 74AHC1G125

Commit message: Update Library
Parts:
- R401, R402: symbol V2_Device:R_0603_220R -> V2_Resistor:0603_220R
Changed lines of the file:
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@@
 		(on_board yes)
 		(dnp no)
-		(property "Reference" "#PWR0404"
+		(property "Reference" "#PWR404"
 			(at 97.79 123.19 0)
 			(effects
@@
 			(project "connect"
 				(path "/6c8448b4-b04d-47e1-934e-e40cbe27a7be/8f187542-ab0c-4216-b848-93c409b6d3f4"
-					(reference "#PWR0404")
+					(reference "#PWR404")
 					(unit 1)
 				)
@@
 		(on_board yes)
 		(dnp no)
-		(property "Reference" "#PWR0406"
+		(property "Reference" "#PWR406"
 			(at 115.57 123.19 0)
 			(effects
@@
 			(project "connect"
 				(path "/6c8448b4-b04d-47e1-934e-e40cbe27a7be/8f187542-ab0c-4216-b848-93c409b6d3f4"
-					(reference "#PWR0406")
-					(unit 1)
-				)
-			)
-		)
-	)
-	(symbol
-		(lib_id "V2_Device:R_0603_220R")
+					(reference "#PWR406")
+					(unit 1)
+				)
+			)
+		)
+	)
+	(symbol
+		(lib_id "V2_Resistor:0603_220R")
 		(at 142.24 109.22 90)
 		(unit 1)
@@
 		(dnp no)
 		(fields_autoplaced yes)
-		(property "Reference" "#PWR0403"
+		(property "Reference" "#PWR403"
 			(at 106.68 105.41 0)
 			(effects
@@
 			(project "connect"
 				(path "/6c8448b4-b04d-47e1-934e-e40cbe27a7be/8f187542-ab0c-4216-b848-93c409b6d3f4"
-					(reference "#PWR0403")
-					(unit 1)
-				)
-			)
-		)
-	)
-	(symbol
-		(lib_id "V2_Device:R_0603_220R")
+					(reference "#PWR403")
+					(unit 1)
+				)
+			)
+		)
+	)
+	(symbol
+		(lib_id "V2_Resistor:0603_220R")
 		(at 154.94 91.44 180)
 		(unit 1)
@@
 		(dnp no)
 		(fields_autoplaced yes)
-		(property "Reference" "#PWR0402"
+		(property "Reference" "#PWR402"
 			(at 180.34 88.9 0)
 			(effects
@@
 			(project "connect"
 				(path "/6c8448b4-b04d-47e1-934e-e40cbe27a7be/8f187542-ab0c-4216-b848-93c409b6d3f4"
-					(reference "#PWR0402")
+					(reference "#PWR402")
 					(unit 1)
 				)
@@
 		(on_board yes)
 		(dnp no)
-		(property "Reference" "#PWR0405"
+		(property "Reference" "#PWR405"
 			(at 106.68 123.19 0)
 			(effects
@@
 			(project "connect"
 				(path "/6c8448b4-b04d-47e1-934e-e40cbe27a7be/8f187542-ab0c-4216-b848-93c409b6d3f4"
-					(reference "#PWR0405")
+					(reference "#PWR405")
 					(unit 1)
 				)
@@
 		(dnp no)
 		(fields_autoplaced yes)
-		(property "Reference" "#PWR0401"
+		(property "Reference" "#PWR401"
 			(at 154.94 92.71 0)
 			(effects
@@
 			(project "connect"
 				(path "/6c8448b4-b04d-47e1-934e-e40cbe27a7be/8f187542-ab0c-4216-b848-93c409b6d3f4"
-					(reference "#PWR0401")
-					(unit 1)
-				)
+					(reference "#PWR401")
+					(unit 1)
+				)
