File: MIDIOut.kicad_sch (KiCad schematic)
At the start: 6 parts, among them J401 SJ2-25404B-SMT-TR, U401 74AHC1G125

Commit message: Update
Parts:
- D401, TVS401: Id (none) -> Diode:${SYMBOL_NAME}
- J401: Id (none) -> Audio:${SYMBOL_NAME}
- R401, R402: Id (none) -> Resistor:${SYMBOL_NAME}
- U401: Id (none) -> 74xGxx:${SYMBOL_NAME}
Changed lines of the file:
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@@
+			)
+		)
+		(property "Id" "Resistor:${SYMBOL_NAME}"
+			(at 156.21 109.22 0)
+			(hide yes)
+			(show_name no)
+			(do_not_autoplace no)
+			(effects
+				(font
+					(size 1.27 1.27)
+				)
 			)
 		)
@@
 			)
 		)
+		(property "Id" "Resistor:${SYMBOL_NAME}"
+			(at 156.21 73.66 0)
+			(hide yes)
+			(show_name no)
+			(do_not_autoplace no)
+			(effects
+				(font
+					(size 1.27 1.27)
+				)
+			)
+		)
 		(pin "1"
 		)
@@
 			)
 		)
+		(property "Id" "Diode:${SYMBOL_NAME}"
+			(at 165.1 92.71 0)
+			(hide yes)
+			(show_name no)
+			(do_not_autoplace no)
+			(effects
+				(font
+					(size 1.27 1.27)
+				)
+			)
+		)
 		(pin "1"
 		)
@@
 		(property "Manufacturer" "Texas Instruments"
 			(at 105.41 132.08 0)
+			(hide yes)
+			(show_name no)
+			(do_not_autoplace no)
+			(effects
+				(font
+					(size 1.27 1.27)
+				)
+			)
+		)
+		(property "Id" "74xGxx:${SYMBOL_NAME}"
+			(at 105.41 121.92 0)
 			(hide yes)
 			(show_name no)
@@
 			)
 		)
+		(property "Id" "Audio:${SYMBOL_NAME}"
+			(at 199.39 127 0)
+			(hide yes)
+			(show_name no)
+			(do_not_autoplace no)
+			(effects
+				(font
+					(size 1.27 1.27)
+				)
+			)
+		)
 		(pin "1"
 		)
@@
 			(hide yes)
 			(show_name no)
+			(do_not_autoplace no)
+			(effects
+				(font
+					(size 1.27 1.27)
+				)
+			)
+		)
+		(property "Id" "Diode:${SYMBOL_NAME}"
+			(at 121.92 113.03 0)
+			(hide yes)
+			(show_name no)

Commit message: Update
Parts:
- renumbered R402 to R401, R401 to R402
Changed lines of the file:
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@@
 		(rev "2026-03-28")
 		(company "Versio Duo")
+		(comment 1 "V2 Link Connector")
 	)
 	(text "﻿Open Collector switching to ignore short-cicuiting.\n\nThe output enters a high impedance state when \nHIGH-level is applied to the output enable (OE) pin."
@@
 		(in_pos_files yes)
 		(dnp no)
-		(property "Reference" "#PWR404"
+		(property "Reference" "#PWR0401"
 			(at 97.79 123.19 0)
 			(hide yes)
@@
 			(project "connect"
 				(path "/6c8448b4-b04d-47e1-934e-e40cbe27a7be/8f187542-ab0c-4216-b848-93c409b6d3f4"
-					(reference "#PWR404")
+					(reference "#PWR0401")
 					(unit 1)
 				)
@@
 		(in_pos_files yes)
 		(dnp no)
-		(property "Reference" "#PWR406"
+		(property "Reference" "#PWR0404"
 			(at 115.57 123.19 0)
 			(hide yes)
@@
 			(project "connect"
 				(path "/6c8448b4-b04d-47e1-934e-e40cbe27a7be/8f187542-ab0c-4216-b848-93c409b6d3f4"
-					(reference "#PWR406")
+					(reference "#PWR0404")
 					(unit 1)
 				)
@@
 		(in_pos_files yes)
 		(dnp no)
-		(property "Reference" "R402"
+		(property "Reference" "R401"
 			(at 142.24 113.03 90)
 			(show_name no)
@@
 			(project "connect"
 				(path "/6c8448b4-b04d-47e1-934e-e40cbe27a7be/8f187542-ab0c-4216-b848-93c409b6d3f4"
-					(reference "R402")
+					(reference "R401")
 					(unit 1)
 				)
@@
 		(dnp no)
 		(fields_autoplaced yes)
-		(property "Reference" "#PWR403"
+		(property "Reference" "#PWR0402"
 			(at 106.68 105.41 0)
 			(hide yes)
@@
 			(project "connect"
 				(path "/6c8448b4-b04d-47e1-934e-e40cbe27a7be/8f187542-ab0c-4216-b848-93c409b6d3f4"
-					(reference "#PWR403")
+					(reference "#PWR0402")
 					(unit 1)
 				)
@@
 		(in_pos_files yes)
 		(dnp no)
-		(property "Reference" "R401"
+		(property "Reference" "R402"
 			(at 162.56 86.36 0)
 			(show_name no)
@@
 			(project "connect"
 				(path "/6c8448b4-b04d-47e1-934e-e40cbe27a7be/8f187542-ab0c-4216-b848-93c409b6d3f4"
-					(reference "R401")
+					(reference "R402")
 					(unit 1)
 				)
@@
 		(dnp no)
 		(fields_autoplaced yes)
-		(property "Reference" "#PWR402"
+		(property "Reference" "#PWR0406"
 			(at 180.34 88.9 0)
 			(hide yes)
@@
 			(project "connect"
 				(path "/6c8448b4-b04d-47e1-934e-e40cbe27a7be/8f187542-ab0c-4216-b848-93c409b6d3f4"
-					(reference "#PWR402")
+					(reference "#PWR0406")
 					(unit 1)
 				)
@@
 		(in_pos_files yes)
 		(dnp no)
-		(property "Reference" "#PWR405"
+		(property "Reference" "#PWR0403"
 			(at 106.68 123.19 0)
 			(hide yes)
@@
 			(project "connect"
 				(path "/6c8448b4-b04d-47e1-934e-e40cbe27a7be/8f187542-ab0c-4216-b848-93c409b6d3f4"
-					(reference "#PWR405")
+					(reference "#PWR0403")
 					(unit 1)
 				)
@@
 		(dnp no)
 		(fields_autoplaced yes)
-		(property "Reference" "#PWR401"
+		(property "Reference" "#PWR0405"
 			(at 156.21 88.9 0)
 			(hide yes)
@@
 			(project "connect"
 				(path "/6c8448b4-b04d-47e1-934e-e40cbe27a7be/8f187542-ab0c-4216-b848-93c409b6d3f4"
-					(reference "#PWR401")
+					(reference "#PWR0405")
 					(unit 1)
 				)

Commit message: Update
Parts:
- added C401: 0u1, V2_Capacitor_SMD:C_0603, symbol V2_Capacitor:0603_0u1
- J401: Rating (none) -> 2.5mm
- U401: Rating (none) -> 8mA
Connections:
- net +5V: now also C401.1
- net GND: now also C401.2
