File: connect.kicad_pcb (KiCad board)
At the start: 4 copper layers, 80 x 34.5 mm, 81 parts, among them J101 Cortex_Debug, J102 DX07S016JA3, J201 NE8FAH, J301 SJ2-25404B-SMT-TR, J401 SJ2-25404B-SMT-TR, SW101 SKSG, SW102 SKSG, SW103 SKSG, SW104 SKSG, SW105 SKSG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

Commit message: Update library
Parts:
- J101: value Cortex_Debug -> Cortex; footprint V2_Cortex_Debug:Cortex_Debug_Pad -> V2_Connector_Debug:Cortex
- U1201: value TPSM33625 -> TPSM365R6FRDNR; footprint V2_Converter_DCDC:TPSM33625 -> V2_Converter_DCDC:QFN-11
Routing:
- net /SWCLK: track 7.86 -> 16.4 mm, vias 2 -> 0
- net +3V3: track 132.7 -> 136.5 mm, vias 13 -> 12
- net GND: track 72.6 -> 72.5 mm, vias 108 -> 106

Commit message: Use date as revision
Other:
- board text added: "2026-02-07 stencil"
Changed lines of the file:
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@@
 	(title_block
 		(date "2026-02-10")
-		(rev "2026-02-10")
+		(rev "2026-02-07")
 	)
 	(layers
@@
 		(layer "F.Fab")
 	)
+	(gr_text "2026-02-07 stencil\n"
+		(at 62.5 80 0)
+		(layer "F.Fab")
+		(effects
+			(font
+				(size 0.5 0.5)
+				(thickness 0.0625)
+			)
+			(justify left bottom)
+		)
+	)
 	(segment

Commit message: Replace Order_Number
Parts:
- INFO101: value Order_Number -> ~; footprint V2_Production:Order_Number -> V2_Production:Revision
Changed lines of the file:
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@@
 		)
 	)
-	(property "Order-Number" "JLCJLCJLCJLC")
 	(net 0 "")
 	(net 1 "GND")
@@
 	(net 110 "unconnected-(U102-PA09-Pad18)")
 	(net 111 "/Button-4")
-	(net 112 "unconnected-(J401-R2-Pad4)_2")
-	(net 113 "unconnected-(J401-SW-Pad10)_1")
-	(net 114 "unconnected-(J301-R2-Pad4)_2")
-	(net 115 "unconnected-(J301-SW-Pad10)_1")
+	(net 112 "unconnected-(J401-R2-Pad4)_1")
+	(net 113 "unconnected-(J401-SW-Pad10)")
+	(net 114 "unconnected-(J301-R2-Pad4)")
+	(net 115 "unconnected-(J301-SW-Pad10)")
 	(footprint "V2_LED:WS2812-2020"
 		(layer "F.Cu")
@@
 			(keep_end_layers yes)
 			(zone_layer_connections)
-			(net 112 "unconnected-(J401-R2-Pad4)_2")
+			(net 112 "unconnected-(J401-R2-Pad4)_1")
 			(pinfunction "R2")
 			(pintype "passive+no_connect")
@@
 			(keep_end_layers yes)
 			(zone_layer_connections)
-			(net 112 "unconnected-(J401-R2-Pad4)_2")
+			(net 112 "unconnected-(J401-R2-Pad4)_1")
 			(pinfunction "R2")
 			(pintype "passive+no_connect")
@@
 			(layers "F.Cu")
 			(roundrect_rratio 0.1)
-			(net 112 "unconnected-(J401-R2-Pad4)_2")
+			(net 112 "unconnected-(J401-R2-Pad4)_1")
 			(pinfunction "R2")
 			(pintype "passive+no_connect")
@@
 			(keep_end_layers yes)
 			(zone_layer_connections)
-			(net 113 "unconnected-(J401-SW-Pad10)_1")
+			(net 113 "unconnected-(J401-SW-Pad10)")
 			(pinfunction "SW")
 			(pintype "passive+no_connect")
@@
 			(layers "F.Cu")
 			(roundrect_rratio 0.2)
-			(net 113 "unconnected-(J401-SW-Pad10)_1")
+			(net 113 "unconnected-(J401-SW-Pad10)")
 			(pinfunction "SW")
 			(pintype "passive+no_connect")
@@
 		)
 	)
-	(footprint "V2_Production:Order_Number"
+	(footprint "V2_Production:Revision"
 		(layer "F.Cu")
 		(at 102.5 116.25)
@@
 			)
 		)
-		(property "Value" "Order_Number"
+		(property "Value" "~"
 			(at 0 2.27 0)
 			(unlocked yes)
@@
 		(sheetname "/")
 		(sheetfile "connect.kicad_sch")
-		(attr exclude_from_pos_files exclude_from_bom)
-		(fp_rect
-			(start -7 -0.75)
-			(end 7 0.75)
-			(stroke
-				(width 0.05)
-				(type default)
+		(attr exclude_from_pos_files exclude_from_bom allow_missing_courtyard)
+		(fp_text user "${REVISION} – ${ISSUE_DATE}"
+			(at 0 0 0)
+			(unlocked yes)
+			(layer "F.SilkS")
+			(effects
+				(font
+					(size 0.6 0.6)
+					(thickness 0.06)
+				)
 			)
-			(fill no)
-			(layer "F.CrtYd")
 		)
-		(fp_text user "${Order-Number}"
+		(fp_text user "${REVISION} – ${ISSUE_DATE}"
 			(at 0 0 0)
 			(unlocked yes)
-			(layer "F.SilkS")
+			(layer "F.Fab")
 			(effects
 				(font
-					(size 0.8 0.8)
-					(thickness 0.12)
+					(size 0.6 0.6)
+					(thickness 0.06)
 				)
 			)
@@
 			)
 		)
-		(property "Sim.Enable" "0"
-			(at 0 0 0)
-			(unlocked yes)
-			(layer "F.Fab")
-			(hide yes)
-			(effects
-				(font
-					(size 1 1)
-					(thickness 0.15)
-				)
-			)
-		)
 		(sheetname "/")
 		(sheetfile "connect.kicad_sch")
@@
 			)
 		)
+		(pad "" smd roundrect
+			(at -1.25 0 90)
+			(size 1 1.8)
+			(layers "F.Paste")
+			(roundrect_rratio 0.1)
+			(chamfer_ratio 0.3)
+			(chamfer top_right bottom_right)
+		)
+		(pad "" smd roundrect
+			(at 1.25 0 90)
+			(size 1 1.8)
+			(layers "F.Paste")
+			(roundrect_rratio 0.1)
+			(chamfer_ratio 0.3)
+			(chamfer top_left bottom_left)
+		)
 		(pad "1" smd roundrect
 			(at 1.25 0 90)
 			(size 1 1.8)
-			(layers "F.Cu" "F.Mask" "F.Paste")
-			(roundrect_rratio 0.15)
+			(layers "F.Cu" "F.Mask")
+			(roundrect_rratio 0.1)
 			(net 20 "/XOUT32")
 			(pinfunction "1")
@@
 			(at -1.25 0 90)
 			(size 1 1.8)
-			(layers "F.Cu" "F.Mask" "F.Paste")
-			(roundrect_rratio 0.15)
+			(layers "F.Cu" "F.Mask")
+			(roundrect_rratio 0.1)
 			(net 17 "/XIN32")
 			(pinfunction "2")
@@
 			(keep_end_layers yes)
 			(zone_layer_connections)
-			(net 114 "unconnected-(J301-R2-Pad4)_2")
+			(net 114 "unconnected-(J301-R2-Pad4)")
 			(pinfunction "R2")
 			(pintype "passive+no_connect")
@@
 			(keep_end_layers yes)
 			(zone_layer_connections)
-			(net 114 "unconnected-(J301-R2-Pad4)_2")
+			(net 114 "unconnected-(J301-R2-Pad4)")
 			(pinfunction "R2")
 			(pintype "passive+no_connect")
@@
 			(layers "F.Cu")
 			(roundrect_rratio 0.1)
-			(net 114 "unconnected-(J301-R2-Pad4)_2")
+			(net 114 "unconnected-(J301-R2-Pad4)")
 			(pinfunction "R2")
 			(pintype "passive+no_connect")
@@
 			(keep_end_layers yes)
 			(zone_layer_connections)
-			(net 115 "unconnected-(J301-SW-Pad10)_1")
+			(net 115 "unconnected-(J301-SW-Pad10)")
 			(pinfunction "SW")
 			(pintype "passive+no_connect")
@@
 			(layers "F.Cu")
 			(roundrect_rratio 0.2)
-			(net 115 "unconnected-(J301-SW-Pad10)_1")
+			(net 115 "unconnected-(J301-SW-Pad10)")
 			(pinfunction "SW")
 			(pintype "passive+no_connect")

Commit message: Update Library
Parts:
- C1203, C1204: value 22u -> 10u

Commit message: Update
Connections:
- net /VBUS renamed /+VBUS

Commit message: Update
Parts:
- C1203, C1204: value 10u -> 22u
Changed lines of the file:
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@@
 			)
 		)
-		(property "Value" "10u"
+		(property "Value" "22u"
 			(at 0 2.3 180)
 			(layer "F.Fab")
@@
 			)
 		)
-		(property "Value" "10u"
+		(property "Value" "22u"
 			(at 0 2.3 180)
 			(layer "F.Fab")

Commit message: Refresh
Connections:
- net /+VBUS renamed +VBUS
