File: connect.kicad_pcb (KiCad board)
At the start: 4 copper layers, 80 x 34.5 mm, 81 parts, among them J101 Cortex, J102 DX07S016JA3, J201 NE8FAH, J301 SJ2-25404B-SMT-TR, J401 SJ2-25404B-SMT-TR, SW101 SKSG, SW102 SKSG, SW103 SKSG, SW104 SKSG, SW105 SKSG, U101 TPS78433QWDRBRQ1, U102 ATSAMD51J, U1201 TPSM365R6FRDNR, U201 THVD2442, U301 TLP2361, U401 74AHC1G125, Y101 32k768

Commit message: Replace step-down
Parts:
- removed R1201: 40k2, V2_Resistor_SMD:R_0603
- removed R1202: 10k, V2_Resistor_SMD:R_0603
- U1201: value TPSM365R6FRDNR -> TPSM33620S5QRDNRQ1
- turned C1205 to 0 degrees
Connections:
- C1205 pad 1: /Power +5V/Vcc -> GND
- C1205 pad 2: GND -> /Power +5V/Vcc
- U1201 pad 11: /Power +5V/Vcc -> GND
- U1201 pad 9: /Power +5V/Feedback -> /+5V-Link
Routing:
- net /Power +5V/Vcc: track 9.70 -> 1.64 mm
- net /Power +5V/Feedback: track 3.11 -> 0.00 mm
- net /+5V-Link: track 12.3 -> 14.8 mm
- net GND: vias 108 -> 110

Commit message: Update
Routing:
- net GND: vias 110 -> 111

Commit message: Update
Parts:
- renumbered C107 to C101, C110 to C102, C101 to C103, C102 to C104, C103 to C105, C104 to C106, C105 to C107, C106 to C108, C108 to C109, C111 to C110, C109 to C111, C302 to C301, C301 to C302, C1201 to C601, C1202 to C602, C1205 to C603, C1203 to C604, C1204 to C605, D104 to D102, D102 to D103, D103 to D104, D505 to D502, D509 to D503, D513 to D504, D517 to D505, D502 to D506, D506 to D507, D510 to D508, D514 to D509, D518 to D510, D503 to D511, D507 to D512, D511 to D513, D515 to D514, D519 to D515, D504 to D516, D508 to D517, D512 to D518, D516 to D519, R104 to R101, R101 to R102, R102 to R103, R103 to R104, R402 to R401, R401 to R402, SW105 to SW101, SW101 to SW102, SW102 to SW103, SW103 to SW104, SW104 to SW105, U102 to U101, U101 to U102, U1201 to U601
Connections:
- net /+VDDCORE renamed /+VCORE

Commit message: Update
Parts:
- added C401: 0u1, V2_Capacitor_SMD:C_0603, F.Cu at (121.5, 111.5)
- moved U401 0.75 mm to (121.5, 114.0)
