File: LEDs.kicad_sch (KiCad schematic)
At the start: 20 parts

Commit message: Refresh
Other:
- title: DMX LED -> V2 connect
Changed lines of the file:
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@@
 	(paper "A4")
 	(title_block
-		(title "DMX LED")
-		(date "2026-03-24")
+		(title "V2 connect")
+		(date "2026-03-26")
 		(rev "2026-03-14")
 		(company "Versio Duo")
