File: PowerSupply.kicad_sch (KiCad schematic)
At the start: 8 parts, among them U1201 TPSM33625

Commit message: Update library
Parts:
- U1201: value TPSM33625 -> TPSM365R6FRDNR; footprint V2_Converter_DCDC:TPSM33625 -> V2_Converter_DCDC:QFN-11; symbol V2_Converter_DCDC:TPSM33625 -> V2_Converter_DCDC:TPSM365R6FRDNR; Mouser 595-TPSM33625RDNR -> 595-TPSM365R6FRDNR; Product TPSM33625RDNR -> TPSM365R6FRDNR; Rating (none) -> 600mA
Changed lines of the file:
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@@
 	)
 	(symbol
-		(lib_id "V2_Converter_DCDC:TPSM33625")
+		(lib_id "V2_Converter_DCDC:TPSM365R6FRDNR")
 		(at 148.59 102.87 0)
 		(unit 1)
@@
 		(dnp no)
 		(property "Reference" "U1201"
-			(at 141.986 87.63 0)
+			(at 141.986 87.122 0)
 			(effects
 				(font
@@
 			)
 		)
-		(property "Value" "TPSM33625"
-			(at 144.78 90.17 0)
+		(property "Value" "TPSM365R6FRDNR"
+			(at 138.43 90.17 0)
 			(effects
 				(font
 					(size 1.524 1.524)
 				)
+				(justify left)
 			)
 		)
-		(property "Footprint" "V2_Converter_DCDC:TPSM33625"
-			(at 148.59 118.11 0)
+		(property "Footprint" "V2_Converter_DCDC:QFN-11"
+			(at 148.59 140.97 0)
 			(effects
 				(font
@@
 			)
 		)
-		(property "Datasheet" "https://www.ti.com/lit/ds/symlink/tpsm33625.pdf"
-			(at 153.67 118.11 0)
+		(property "Datasheet" ""
+			(at 148.59 143.51 0)
 			(effects
 				(font
@@
 			)
 		)
-		(property "Mouser" "595-TPSM33625RDNR"
+		(property "Mouser" "595-TPSM365R6FRDNR"
 			(at 148.59 151.13 0)
+			(show_name yes)
 			(effects
 				(font
@@
 		(property "Manufacturer" "Texas Instruments"
 			(at 148.59 146.05 0)
+			(show_name yes)
 			(effects
 				(font
@@
 			)
 		)
-		(property "Product" "TPSM33625RDNR"
+		(property "Product" "TPSM365R6FRDNR"
 			(at 148.59 148.59 0)
+			(show_name yes)
 			(effects
 				(font
+					(size 1.27 1.27)
+				)
+				(hide yes)
+			)
+		)
+		(property "Rating" "600mA"
+			(at 148.59 153.67 0)
+			(effects
+				(font

Commit message: Update Library
Parts:
- C1201: symbol V2_Device:C_1210_10u -> V2_Capacitor:1210_10u
- C1202: symbol V2_Device:C_0603_0u1 -> V2_Capacitor:0603_0u1
- C1203, C1204: value 22u -> 10u; symbol V2_Device:C_1210_22u -> V2_Capacitor:1210_22u
- C1205: symbol V2_Device:C_0603_1u -> V2_Capacitor:0603_1u
- R1201: symbol V2_Device:R_0603_40k2 -> V2_Resistor:0603_40k2
- R1202: symbol V2_Device:R_0603_10k -> V2_Resistor:0603_10k
Changed lines of the file:
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@@
 	)
 	(symbol
-		(lib_id "V2_Device:C_0603_0u1")
+		(lib_id "V2_Capacitor:0603_0u1")
 		(at 109.22 97.79 0)
 		(unit 1)
@@
 	)
 	(symbol
-		(lib_id "V2_Device:C_1210_22u")
+		(lib_id "V2_Capacitor:1210_22u")
 		(at 195.58 97.79 0)
 		(unit 1)
@@
 			)
 		)
-		(property "Value" "22u"
+		(property "Value" "10u"
 			(at 198.12 99.06 0)
 			(effects
@@
 	)
 	(symbol
-		(lib_id "V2_Device:R_0603_40k2")
+		(lib_id "V2_Resistor:0603_40k2")
 		(at 172.72 97.79 0)
 		(unit 1)
@@
 		(on_board yes)
 		(dnp no)
-		(property "Reference" "#PWR01203"
+		(property "Reference" "#PWR1203"
 			(at 185.42 106.68 0)
 			(effects
@@
 			(project "connect"
 				(path "/6c8448b4-b04d-47e1-934e-e40cbe27a7be/095cddf1-6522-4d3b-885d-b21acd91d0c6"
-					(reference "#PWR01203")
+					(reference "#PWR1203")
 					(unit 1)
 				)
@@
 		(on_board yes)
 		(dnp no)
-		(property "Reference" "#PWR01204"
+		(property "Reference" "#PWR1204"
 			(at 195.58 106.68 0)
 			(effects
@@
 			(project "connect"
 				(path "/6c8448b4-b04d-47e1-934e-e40cbe27a7be/095cddf1-6522-4d3b-885d-b21acd91d0c6"
-					(reference "#PWR01204")
+					(reference "#PWR1204")
 					(unit 1)
 				)
@@
 		(on_board yes)
 		(dnp no)
-		(property "Reference" "#PWR01201"
+		(property "Reference" "#PWR1201"
 			(at 97.79 106.68 0)
 			(effects
@@
 			(project "connect"
 				(path "/6c8448b4-b04d-47e1-934e-e40cbe27a7be/095cddf1-6522-4d3b-885d-b21acd91d0c6"
-					(reference "#PWR01201")
+					(reference "#PWR1201")
 					(unit 1)
 				)
@@
 		(on_board yes)
 		(dnp no)
-		(property "Reference" "#PWR01205"
+		(property "Reference" "#PWR1205"
 			(at 172.72 111.76 0)
 			(effects
@@
 			(project "connect"
 				(path "/6c8448b4-b04d-47e1-934e-e40cbe27a7be/095cddf1-6522-4d3b-885d-b21acd91d0c6"
-					(reference "#PWR01205")
+					(reference "#PWR1205")
 					(unit 1)
 				)
@@
 		(on_board yes)
 		(dnp no)
-		(property "Reference" "#PWR01202"
+		(property "Reference" "#PWR1202"
 			(at 109.22 106.68 0)
 			(effects
@@
 			(project "connect"
 				(path "/6c8448b4-b04d-47e1-934e-e40cbe27a7be/095cddf1-6522-4d3b-885d-b21acd91d0c6"
-					(reference "#PWR01202")
-					(unit 1)
-				)
-			)
-		)
-	)
-	(symbol
-		(lib_id "V2_Device:C_0603_1u")
+					(reference "#PWR1202")
+					(unit 1)
+				)
+			)
+		)
+	)
+	(symbol
+		(lib_id "V2_Capacitor:0603_1u")
 		(at 128.27 107.95 0)
 		(unit 1)
@@
 	)
 	(symbol
-		(lib_id "V2_Device:C_1210_22u")
+		(lib_id "V2_Capacitor:1210_22u")
 		(at 185.42 97.79 0)
 		(unit 1)
@@
 			)
 		)
-		(property "Value" "22u"
+		(property "Value" "10u"
 			(at 187.96 98.806 0)
 			(effects
@@
 		(on_board yes)
 		(dnp no)
-		(property "Reference" "#PWR01206"
+		(property "Reference" "#PWR1206"
 			(at 128.27 116.84 0)
 			(effects
@@
 			(project "connect"
 				(path "/6c8448b4-b04d-47e1-934e-e40cbe27a7be/095cddf1-6522-4d3b-885d-b21acd91d0c6"
-					(reference "#PWR01206")
-					(unit 1)
-				)
-			)
-		)
-	)
-	(symbol
-		(lib_id "V2_Device:R_0603_10k")
+					(reference "#PWR1206")
+					(unit 1)
+				)
+			)
+		)
+	)
+	(symbol
+		(lib_id "V2_Resistor:0603_10k")
 		(at 172.72 102.87 0)
 		(unit 1)
@@
 		(on_board yes)
 		(dnp no)
-		(property "Reference" "#PWR01207"
+		(property "Reference" "#PWR1207"
 			(at 148.59 121.92 0)
 			(effects
@@
 			(project "connect"
 				(path "/6c8448b4-b04d-47e1-934e-e40cbe27a7be/095cddf1-6522-4d3b-885d-b21acd91d0c6"
-					(reference "#PWR01207")
-					(unit 1)
-				)
-			)
-		)
-	)
-	(symbol
-		(lib_id "V2_Device:C_1210_10u")
+					(reference "#PWR1207")
+					(unit 1)
+				)
+			)
+		)
+	)
+	(symbol
+		(lib_id "V2_Capacitor:1210_10u")
 		(at 97.79 97.79 0)
 		(unit 1)

Commit message: Update
Parts:
- C1203, C1204: value 10u -> 22u
Changed lines of the file:
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@@
 			)
 		)
-		(property "Value" "10u"
+		(property "Value" "22u"
 			(at 198.12 99.06 0)
 			(effects
@@
 			)
 		)
-		(property "Value" "10u"
+		(property "Value" "22u"
 			(at 187.96 98.806 0)
 			(effects

Commit message: Export stencil
Parts:
- C1201: Mouser 810-CNA6P1X7R1H106K2 -> 810-CNC6P1X7R1H106K2; Product CNA6P1X7R1H106K250AE -> CNC6P1X7R1H106K250AE
Changed lines of the file:
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@@
 			)
 		)
-		(property "Mouser" "810-CNA6P1X7R1H106K2"
+		(property "Mouser" "810-CNC6P1X7R1H106K2"
 			(at 97.79 120.65 0)
 			(show_name yes)
@@
 			)
 		)
-		(property "Product" "CNA6P1X7R1H106K250AE"
+		(property "Product" "CNC6P1X7R1H106K250AE"
 			(at 97.79 115.57 0)
 			(show_name yes)

Commit message: KiCad 10
Other:
- company: +5V -> Versio Duo

Commit message: Refresh
Other:
- title: Power Supply -> V2 connect
Changed lines of the file:
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@@
 	(paper "A4")
 	(title_block
-		(title "Power Supply")
-		(date "2026-03-24")
+		(title "V2 connect")
+		(date "2026-03-26")
 		(rev "2026-03-14")
 		(company "Versio Duo")
