File: connect.kicad_sch (KiCad schematic)
At the start: 37 parts, among them J101 Cortex, J102 DX07S016JA3, SW101 SKSG, SW102 SKSG, SW103 SKSG, SW104 SKSG, SW105 SKSG, U101 TPS78433QWDRBRQ1, U102 ATSAMD51J, Y101 32k768

Commit message: Refresh
Parts:
- C107, C110: Rating (none) -> 50V
- SW101, SW102, SW103, SW104, SW105: Rating (none) -> 1.6N
Changed lines of the file:
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@@
 			)
 		)
+		(property "Rating" "1.6N"
+			(at 264.16 44.45 0)
+			(hide yes)
+			(show_name no)
+			(do_not_autoplace no)
+			(effects
+				(font
+					(size 1.27 1.27)
+				)
+			)
+		)
 		(pin "1"
 		)
@@
 			)
 		)
+		(property "Rating" "50V"
+			(at -1.27 43.18 0)
+			(hide yes)
+			(show_name no)
+			(do_not_autoplace no)
+			(effects
+				(font
+					(size 1.27 1.27)
+				)
+			)
+		)
 		(pin "1"
 		)
@@
 			)
 		)
+		(property "Rating" "1.6N"
+			(at 264.16 78.74 0)
+			(hide yes)
+			(show_name no)
+			(do_not_autoplace no)
+			(effects
+				(font
+					(size 1.27 1.27)
+				)
+			)
+		)
 		(pin "1"
 		)
@@
 			)
 		)
+		(property "Rating" "50V"
+			(at -1.27 38.1 0)
+			(hide yes)
+			(show_name no)
+			(do_not_autoplace no)
+			(effects
+				(font
+					(size 1.27 1.27)
+				)
+			)
+		)
 		(pin "1"
 		)
@@
 			)
 		)
+		(property "Rating" "1.6N"
+			(at 133.35 96.52 0)
+			(hide yes)
+			(show_name no)
+			(do_not_autoplace no)
+			(effects
+				(font
+					(size 1.27 1.27)
+				)
+			)
+		)
 		(pin "1"
 		)
@@
 			)
 		)
+		(property "Rating" "1.6N"
+			(at 264.16 67.31 0)
+			(hide yes)
+			(show_name no)
+			(do_not_autoplace no)
+			(effects
+				(font
+					(size 1.27 1.27)
+				)
+			)
+		)
 		(pin "1"
 		)
@@
 			(hide yes)
 			(show_name no)
+			(do_not_autoplace no)
+			(effects
+				(font
+					(size 1.27 1.27)
+				)
+			)
+		)
+		(property "Rating" "1.6N"
+			(at 264.16 55.88 0)
+			(hide yes)
+			(show_name no)

Commit message: Update
Parts:
- C101, C102, C103, C104, C105, C106, C107, C108, C109, C110, C111: Id (none) -> Capacitor:${SYMBOL_NAME}
- D101: Id (none) -> LED:${SYMBOL_NAME}
- D102, D103, D104, TVS101: Id (none) -> Diode:${SYMBOL_NAME}
- ESD101: Id (none) -> ESD:${SYMBOL_NAME}
- J102: Id (none) -> USB:${SYMBOL_NAME}
- R101, R102, R103, R104: Id (none) -> Resistor:${SYMBOL_NAME}
- SW101, SW102, SW103, SW104, SW105: Id (none) -> Button:${SYMBOL_NAME}
- U101: Id (none) -> LDO:${SYMBOL_NAME}
- U102: Id (none) -> MCU:${SYMBOL_NAME}
- Y101: Id (none) -> Crystal:${SYMBOL_NAME}

Commit message: Update
Parts:
- D101: Rating (none) -> 605nm
- J102: Rating (none) -> USB2.0
- U101: Rating (none) -> 300mA
- Y101: Rating (none) -> 10ppm
Changed lines of the file:
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@@
 			)
 		)
+		(property "Rating" "300mA"
+			(at 186.69 91.44 0)
+			(hide yes)
+			(show_name no)
+			(do_not_autoplace no)
+			(effects
+				(font
+					(size 1.27 1.27)
+				)
+			)
+		)
 		(pin "1"
 		)
@@
 			)
 		)
+		(property "Rating" "10ppm"
+			(at 44.45 40.64 0)
+			(hide yes)
+			(show_name no)
+			(do_not_autoplace no)
+			(effects
+				(font
+					(size 1.27 1.27)
+				)
+			)
+		)
 		(pin "1"
 		)
@@
 			)
 		)
-		(property "Sim.Pins" "1=K 2=A"
-			(at 132.08 58.42 0)
+		(property "Mouser" "755-SML-D12D1WT86"
+			(at 132.08 66.04 0)
 			(hide yes)
 			(show_name no)
@@
 			)
 		)
-		(property "Mouser" "755-SML-D12D1WT86"
-			(at 132.08 66.04 0)
+		(property "Product" "SML-D12D1WT86"
+			(at 132.08 71.12 0)
 			(hide yes)
 			(show_name no)
@@
 			)
 		)
-		(property "Product" "SML-D12D1WT86"
-			(at 132.08 71.12 0)
+		(property "Manufacturer" "ROHM Semiconductor "
+			(at 132.08 68.58 0)
 			(hide yes)
 			(show_name no)
@@
 			)
 		)
-		(property "Manufacturer" "ROHM Semiconductor "
-			(at 132.08 68.58 0)
+		(property "Id" "LED:${SYMBOL_NAME}"
+			(at 132.08 63.5 0)
 			(hide yes)
 			(show_name no)
@@
 			)
 		)
-		(property "Id" "LED:${SYMBOL_NAME}"
-			(at 132.08 63.5 0)
+		(property "Rating" "605nm"
+			(at 132.08 76.2 0)
 			(hide yes)
 			(show_name no)
@@
 			(hide yes)
 			(show_name no)
+			(do_not_autoplace no)
+			(effects
+				(font
+					(size 1.27 1.27)
+				)
+			)
+		)
+		(property "Rating" "USB2.0"
+			(at 176.53 140.97 0)
+			(hide yes)
+			(show_name no)

Commit message: Update
Parts:
- renumbered C107 to C101, C110 to C102, C101 to C103, C102 to C104, C103 to C105, C104 to C106, C105 to C107, C106 to C108, C108 to C109, C111 to C110, C109 to C111, D104 to D102, D102 to D103, D103 to D104, R104 to R101, R101 to R102, R102 to R103, R103 to R104, SW105 to SW101, SW101 to SW102, SW102 to SW103, SW103 to SW104, SW104 to SW105, U102 to U101, U101 to U102
Connections:
- net +VDDCORE renamed +VCORE

Commit message: Update
Parts:
- ESD101: Rating (none) -> 20kV
- U101: Rating (none) -> Cortex-M4F
