File: hardware/plug/MIDIOut.kicad_sch (KiCad schematic)
At the start: 7 parts, among them J301 SJ2-25404B-SMT-TR, U301 74AHC1G125

Commit message: Good Bye Imperial
Parts:
- C301: footprint V2_Capacitor_SMD:C_0603 -> V2_Capacitor_SMD:C_1608; symbol V2_Capacitor:0603_0u1 -> V2_Capacitor:1608_0u1
- R301, R302: footprint V2_Resistor_SMD:R_0603 -> V2_Resistor_SMD:R_1608; symbol V2_Resistor:0603_220R -> V2_Resistor:1608_220R
- TVS301: footprint V2_Diode_SMD:D_0603 -> V2_Diode_SMD:D_1608

Commit message: Refresh
Parts:
- renumbered C301 to C501, D301 to D501, J301 to J501, R301 to R501, R302 to R502, TVS301 to TVS501, U301 to U501
Changed lines of the file:
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@@
 		(in_pos_files yes)
 		(dnp no)
-		(property "Reference" "C301"
+		(property "Reference" "C501"
 			(at 114.3 85.09 0)
 			(show_name no)
@@
 		)
 		(property "LCSC" ""
-			(at 106.68 86.36 0)
-			(hide yes)
-			(show_name no)
-			(do_not_autoplace no)
-			(effects
-				(font
-					(size 1.27 1.27)
-				)
-			)
-		)
-		(property "Sim.Enable" ""
 			(at 106.68 86.36 0)
 			(hide yes)
@@
 			(project "plug"
 				(path "/6c8448b4-b04d-47e1-934e-e40cbe27a7be/2737a175-b1a1-4dfd-b186-4741ca8995da"
-					(reference "C301")
+					(reference "C501")
 					(unit 1)
 				)
@@
 		(in_pos_files yes)
 		(dnp no)
-		(property "Reference" "#PWR0301"
+		(property "Reference" "#PWR0501"
 			(at 97.79 123.19 0)
 			(hide yes)
@@
 			(project "plug"
 				(path "/6c8448b4-b04d-47e1-934e-e40cbe27a7be/2737a175-b1a1-4dfd-b186-4741ca8995da"
-					(reference "#PWR0301")
+					(reference "#PWR0501")
 					(unit 1)
 				)
@@
 		(dnp no)
 		(fields_autoplaced yes)
-		(property "Reference" "#PWR0303"
+		(property "Reference" "#PWR0503"
 			(at 106.68 95.25 0)
 			(hide yes)
@@
 			(project "plug"
 				(path "/6c8448b4-b04d-47e1-934e-e40cbe27a7be/2737a175-b1a1-4dfd-b186-4741ca8995da"
-					(reference "#PWR0303")
+					(reference "#PWR0503")
 					(unit 1)
 				)
@@
 		(in_pos_files yes)
 		(dnp no)
-		(property "Reference" "#PWR0306"
+		(property "Reference" "#PWR0506"
 			(at 115.57 123.19 0)
 			(hide yes)
@@
 			(project "plug"
 				(path "/6c8448b4-b04d-47e1-934e-e40cbe27a7be/2737a175-b1a1-4dfd-b186-4741ca8995da"
-					(reference "#PWR0306")
+					(reference "#PWR0506")
 					(unit 1)
 				)
@@
 		(dnp no)
 		(fields_autoplaced yes)
-		(property "Reference" "#PWR0302"
+		(property "Reference" "#PWR0502"
 			(at 106.68 87.63 0)
 			(hide yes)
@@
 			(project "plug"
 				(path "/6c8448b4-b04d-47e1-934e-e40cbe27a7be/2737a175-b1a1-4dfd-b186-4741ca8995da"
-					(reference "#PWR0302")
+					(reference "#PWR0502")
 					(unit 1)
 				)
@@
 		(in_pos_files yes)
 		(dnp no)
-		(property "Reference" "R301"
+		(property "Reference" "R501"
 			(at 142.24 113.03 90)
 			(show_name no)
@@
 		)
 		(property "LCSC" ""
-			(at 142.24 109.22 90)
-			(hide yes)
-			(show_name no)
-			(do_not_autoplace no)
-			(effects
-				(font
-					(size 1.27 1.27)
-				)
-			)
-		)
-		(property "Sim.Enable" ""
 			(at 142.24 109.22 90)
 			(hide yes)
@@
 			(project "plug"
 				(path "/6c8448b4-b04d-47e1-934e-e40cbe27a7be/2737a175-b1a1-4dfd-b186-4741ca8995da"
-					(reference "R301")
+					(reference "R501")
 					(unit 1)
 				)
@@
 		(dnp no)
 		(fields_autoplaced yes)
-		(property "Reference" "#PWR0304"
+		(property "Reference" "#PWR0504"
 			(at 106.68 105.41 0)
 			(hide yes)
@@
 			(project "plug"
 				(path "/6c8448b4-b04d-47e1-934e-e40cbe27a7be/2737a175-b1a1-4dfd-b186-4741ca8995da"
-					(reference "#PWR0304")
+					(reference "#PWR0504")
 					(unit 1)
 				)
@@
 		(in_pos_files yes)
 		(dnp no)
-		(property "Reference" "R302"
+		(property "Reference" "R502"
 			(at 162.56 86.36 0)
 			(show_name no)
@@
 		)
 		(property "LCSC" ""
-			(at 156.21 87.63 0)
-			(hide yes)
-			(show_name no)
-			(do_not_autoplace no)
-			(effects
-				(font
-					(size 1.27 1.27)
-				)
-			)
-		)
-		(property "Sim.Enable" ""
 			(at 156.21 87.63 0)
 			(hide yes)
@@
 			(project "plug"
 				(path "/6c8448b4-b04d-47e1-934e-e40cbe27a7be/2737a175-b1a1-4dfd-b186-4741ca8995da"
-					(reference "R302")
+					(reference "R502")
 					(unit 1)
 				)
@@
 		(dnp no)
 		(fields_autoplaced yes)
-		(property "Reference" "#PWR0308"
+		(property "Reference" "#PWR0508"
 			(at 180.34 88.9 0)
 			(hide yes)
@@
 			(project "plug"
 				(path "/6c8448b4-b04d-47e1-934e-e40cbe27a7be/2737a175-b1a1-4dfd-b186-4741ca8995da"
-					(reference "#PWR0308")
+					(reference "#PWR0508")
 					(unit 1)
 				)
@@
 		(in_pos_files yes)
 		(dnp no)
-		(property "Reference" "#PWR0305"
+		(property "Reference" "#PWR0505"
 			(at 106.68 123.19 0)
 			(hide yes)
@@
 			(project "plug"
 				(path "/6c8448b4-b04d-47e1-934e-e40cbe27a7be/2737a175-b1a1-4dfd-b186-4741ca8995da"
-					(reference "#PWR0305")
+					(reference "#PWR0505")
 					(unit 1)
 				)
@@
 		(in_pos_files yes)
 		(dnp no)
-		(property "Reference" "D301"
+		(property "Reference" "D501"
 			(at 165.1 93.98 90)
 			(show_name no)
@@
 		)
 		(property "LCSC" ""
-			(at 156.21 92.71 90)
-			(hide yes)
-			(show_name no)
-			(do_not_autoplace no)
-			(effects
-				(font
-					(size 1.27 1.27)
-				)
-			)
-		)
-		(property "Sim.Enable" ""
 			(at 156.21 92.71 90)
 			(hide yes)
@@
 			(project "plug"
 				(path "/6c8448b4-b04d-47e1-934e-e40cbe27a7be/2737a175-b1a1-4dfd-b186-4741ca8995da"
-					(reference "D301")
+					(reference "D501")
 					(unit 1)
 				)
@@
 		(in_pos_files yes)
 		(dnp no)
-		(property "Reference" "U301"
+		(property "Reference" "U501"
 			(at 111.76 102.87 0)
 			(show_name no)
@@
 		)
 		(property "LCSC" ""
-			(at 105.41 109.22 0)
-			(hide yes)
-			(show_name no)
-			(do_not_autoplace no)
-			(effects
-				(font
-					(size 1.27 1.27)
-				)
-			)
-		)
-		(property "Sim.Enable" ""
 			(at 105.41 109.22 0)
 			(hide yes)
@@
 			(project "plug"
 				(path "/6c8448b4-b04d-47e1-934e-e40cbe27a7be/2737a175-b1a1-4dfd-b186-4741ca8995da"
-					(reference "U301")
+					(reference "U501")
 					(unit 1)
 				)
@@
 		(dnp no)
 		(fields_autoplaced yes)
-		(property "Reference" "#PWR0307"
+		(property "Reference" "#PWR0507"
 			(at 156.21 88.9 0)
 			(hide yes)
@@
 			(project "plug"
 				(path "/6c8448b4-b04d-47e1-934e-e40cbe27a7be/2737a175-b1a1-4dfd-b186-4741ca8995da"
-					(reference "#PWR0307")
+					(reference "#PWR0507")
 					(unit 1)
 				)
@@
 		(in_pos_files yes)
 		(dnp no)
-		(property "Reference" "J301"
+		(property "Reference" "J501"
 			(at 207.264 81.788 0)
 			(show_name no)
@@
 		)
 		(property "LCSC" ""
-			(at 199.39 99.06 0)
-			(hide yes)
-			(show_name no)
-			(do_not_autoplace no)
-			(effects
-				(font
-					(size 1.27 1.27)
-				)
-			)
-		)
-		(property "Sim.Enable" ""
 			(at 199.39 99.06 0)
 			(hide yes)
@@
 			(project "plug"
 				(path "/6c8448b4-b04d-47e1-934e-e40cbe27a7be/2737a175-b1a1-4dfd-b186-4741ca8995da"
-					(reference "J301")
+					(reference "J501")
 					(unit 1)
 				)
@@
 		(in_pos_files yes)
 		(dnp no)
-		(property "Reference" "TVS301"
+		(property "Reference" "TVS501"
 			(at 118.11 113.03 90)
 			(show_name no)
@@
 		)
 		(property "LCSC" ""
-			(at 115.57 113.03 90)
-			(hide yes)
-			(show_name no)
-			(do_not_autoplace no)
-			(effects
-				(font
-					(size 1.27 1.27)
-				)
-			)
-		)
-		(property "Sim.Enable" ""
 			(at 115.57 113.03 90)
 			(hide yes)
@@
 			(project "plug"
 				(path "/6c8448b4-b04d-47e1-934e-e40cbe27a7be/2737a175-b1a1-4dfd-b186-4741ca8995da"
-					(reference "TVS301")
+					(reference "TVS501")
 					(unit 1)
 				)
