File: hardware/plug/PowerSupply.kicad_sch (KiCad schematic)
At the start: 6 parts, among them U1201 TPSM33620S5QRDNRQ1

Commit message: Good Bye Imperial
Parts:
- C1201: footprint V2_Capacitor_SMD:C_1210 -> V2_Capacitor_SMD:C_3225; symbol V2_Capacitor:1210_10u -> V2_Capacitor:3225_10u
- C1202: footprint V2_Capacitor_SMD:C_0603 -> V2_Capacitor_SMD:C_1608; symbol V2_Capacitor:0603_0u1 -> V2_Capacitor:1608_0u1
- C1203: footprint V2_Capacitor_SMD:C_0603 -> V2_Capacitor_SMD:C_1608; symbol V2_Capacitor:0603_1u -> V2_Capacitor:1608_1u
- C1204, C1205: footprint V2_Capacitor_SMD:C_1210 -> V2_Capacitor_SMD:C_3225; symbol V2_Capacitor:1210_22u -> V2_Capacitor:3225_22u
Changed lines of the file:
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@@
+			)
+		)
+		(property "LCSC" ""
+			(at 148.59 102.87 0)
+			(hide yes)
+			(show_name no)
+			(do_not_autoplace no)
+			(effects
+				(font
+					(size 1.27 1.27)
+				)
+			)
+		)
+		(property "Sim.Enable" ""
+			(at 148.59 102.87 0)
+			(hide yes)
+			(show_name no)
+			(do_not_autoplace no)
+			(effects
+				(font
+					(size 1.27 1.27)
+				)
+			)
+		)
+		(property "Voltage" ""
+			(at 148.59 102.87 0)
+			(hide yes)
+			(show_name no)
+			(do_not_autoplace no)
+			(effects
+				(font
+					(size 1.27 1.27)
+				)
 			)
 		)
@@
 	)
 	(symbol
-		(lib_id "V2_Capacitor:0603_0u1")
+		(lib_id "V2_Capacitor:1608_0u1")
 		(at 109.22 97.79 0)
 		(unit 1)
@@
 			)
 		)
-		(property "Footprint" "V2_Capacitor_SMD:C_0603"
+		(property "Footprint" "V2_Capacitor_SMD:C_1608"
 			(at 109.22 114.808 0)
 			(hide yes)
@@
 		(property "Id" "Capacitor:${SYMBOL_NAME}"
 			(at 109.22 113.03 0)
+			(hide yes)
+			(show_name no)
+			(do_not_autoplace no)
+			(effects
+				(font
+					(size 1.27 1.27)
+				)
+			)
+		)
+		(property "LCSC" ""
+			(at 109.22 97.79 0)
+			(hide yes)
+			(show_name no)
+			(do_not_autoplace no)
+			(effects
+				(font
+					(size 1.27 1.27)
+				)
+			)
+		)
+		(property "Sim.Enable" ""
+			(at 109.22 97.79 0)
+			(hide yes)
+			(show_name no)
+			(do_not_autoplace no)
+			(effects
+				(font
+					(size 1.27 1.27)
+				)
+			)
+		)
+		(property "Voltage" ""
+			(at 109.22 97.79 0)
 			(hide yes)
 			(show_name no)
@@
 	)
 	(symbol
-		(lib_id "V2_Capacitor:1210_22u")
+		(lib_id "V2_Capacitor:3225_22u")
 		(at 195.58 97.79 0)
 		(unit 1)
@@
 			)
 		)
-		(property "Footprint" "V2_Capacitor_SMD:C_1210"
+		(property "Footprint" "V2_Capacitor_SMD:C_3225"
 			(at 195.58 114.808 0)
 			(hide yes)
@@
 		(property "Id" "Capacitor:${SYMBOL_NAME}"
 			(at 195.58 113.03 0)
+			(hide yes)
+			(show_name no)
+			(do_not_autoplace no)
+			(effects
+				(font
+					(size 1.27 1.27)
+				)
+			)
+		)
+		(property "LCSC" ""
+			(at 195.58 97.79 0)
+			(hide yes)
+			(show_name no)
+			(do_not_autoplace no)
+			(effects
+				(font
+					(size 1.27 1.27)
+				)
+			)
+		)
+		(property "Sim.Enable" ""
+			(at 195.58 97.79 0)
+			(hide yes)
+			(show_name no)
+			(do_not_autoplace no)
+			(effects
+				(font
+					(size 1.27 1.27)
+				)
+			)
+		)
+		(property "Voltage" ""
+			(at 195.58 97.79 0)
 			(hide yes)
 			(show_name no)
@@
 	)
 	(symbol
-		(lib_id "V2_Capacitor:0603_1u")
+		(lib_id "V2_Capacitor:1608_1u")
 		(at 125.73 105.41 270)
 		(unit 1)
@@
 			)
 		)
-		(property "Footprint" "V2_Capacitor_SMD:C_0603"
+		(property "Footprint" "V2_Capacitor_SMD:C_1608"
 			(at 108.712 105.41 0)
 			(hide yes)
@@
 		(property "Id" "Capacitor:${SYMBOL_NAME}"
 			(at 110.49 105.41 0)
+			(hide yes)
+			(show_name no)
+			(do_not_autoplace no)
+			(effects
+				(font
+					(size 1.27 1.27)
+				)
+			)
+		)
+		(property "LCSC" ""
+			(at 125.73 105.41 90)
+			(hide yes)
+			(show_name no)
+			(do_not_autoplace no)
+			(effects
+				(font
+					(size 1.27 1.27)
+				)
+			)
+		)
+		(property "Sim.Enable" ""
+			(at 125.73 105.41 90)
+			(hide yes)
+			(show_name no)
+			(do_not_autoplace no)
+			(effects
+				(font
+					(size 1.27 1.27)
+				)
+			)
+		)
+		(property "Voltage" ""
+			(at 125.73 105.41 90)
 			(hide yes)
 			(show_name no)
@@
 	)
 	(symbol
-		(lib_id "V2_Capacitor:1210_22u")
+		(lib_id "V2_Capacitor:3225_22u")
 		(at 185.42 97.79 0)
 		(unit 1)
@@
 			)
 		)
-		(property "Footprint" "V2_Capacitor_SMD:C_1210"
+		(property "Footprint" "V2_Capacitor_SMD:C_3225"
 			(at 185.42 114.808 0)
 			(hide yes)
@@
 		(property "Id" "Capacitor:${SYMBOL_NAME}"
 			(at 185.42 113.03 0)
+			(hide yes)
+			(show_name no)
+			(do_not_autoplace no)
+			(effects
+				(font
+					(size 1.27 1.27)
+				)
+			)
+		)
+		(property "LCSC" ""
+			(at 185.42 97.79 0)
+			(hide yes)
+			(show_name no)
+			(do_not_autoplace no)
+			(effects
+				(font
+					(size 1.27 1.27)
+				)
+			)
+		)
+		(property "Sim.Enable" ""
+			(at 185.42 97.79 0)
+			(hide yes)
+			(show_name no)
+			(do_not_autoplace no)
+			(effects
+				(font
+					(size 1.27 1.27)
+				)
+			)
+		)
+		(property "Voltage" ""
+			(at 185.42 97.79 0)
 			(hide yes)
 			(show_name no)
@@
 	)
 	(symbol
-		(lib_id "V2_Capacitor:1210_10u")
+		(lib_id "V2_Capacitor:3225_10u")
 		(at 97.79 97.79 0)
 		(unit 1)
@@
 			)
 		)
-		(property "Footprint" "V2_Capacitor_SMD:C_1210"
+		(property "Footprint" "V2_Capacitor_SMD:C_3225"
 			(at 97.79 114.808 0)
 			(hide yes)
@@
 			(hide yes)
 			(show_name no)
+			(do_not_autoplace no)
+			(effects
+				(font
+					(size 1.27 1.27)
+				)
+			)
+		)
+		(property "LCSC" ""
+			(at 97.79 97.79 0)
+			(hide yes)
+			(show_name no)
+			(do_not_autoplace no)
+			(effects
+				(font
+					(size 1.27 1.27)
+				)
+			)
+		)
+		(property "Sim.Enable" ""
+			(at 97.79 97.79 0)
+			(hide yes)
+			(show_name no)
+			(do_not_autoplace no)
+			(effects
+				(font
+					(size 1.27 1.27)
+				)
+			)
+		)
+		(property "Voltage" ""
+			(at 97.79 97.79 0)
+			(hide yes)
+			(show_name no)

Commit message: Refresh
Parts:
- renumbered C1201 to C201, C1202 to C202, C1203 to C203, C1204 to C204, C1205 to C205, U1201 to U201
Changed lines of the file:
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@@
 		(in_pos_files yes)
 		(dnp no)
-		(property "Reference" "U1201"
-			(at 141.986 87.63 0)
+		(property "Reference" "U201"
+			(at 140.97 87.63 0)
 			(show_name no)
 			(do_not_autoplace no)
@@
 		)
 		(property "LCSC" ""
-			(at 148.59 102.87 0)
-			(hide yes)
-			(show_name no)
-			(do_not_autoplace no)
-			(effects
-				(font
-					(size 1.27 1.27)
-				)
-			)
-		)
-		(property "Sim.Enable" ""
 			(at 148.59 102.87 0)
 			(hide yes)
@@
 			(project "plug"
 				(path "/6c8448b4-b04d-47e1-934e-e40cbe27a7be/095cddf1-6522-4d3b-885d-b21acd91d0c6"
-					(reference "U1201")
+					(reference "U201")
 					(unit 1)
 				)
@@
 		(in_pos_files yes)
 		(dnp no)
-		(property "Reference" "C1202"
+		(property "Reference" "C202"
 			(at 111.76 96.52 0)
 			(show_name no)
@@
 		)
 		(property "LCSC" ""
-			(at 109.22 97.79 0)
-			(hide yes)
-			(show_name no)
-			(do_not_autoplace no)
-			(effects
-				(font
-					(size 1.27 1.27)
-				)
-			)
-		)
-		(property "Sim.Enable" ""
 			(at 109.22 97.79 0)
 			(hide yes)
@@
 			(project "plug"
 				(path "/6c8448b4-b04d-47e1-934e-e40cbe27a7be/095cddf1-6522-4d3b-885d-b21acd91d0c6"
-					(reference "C1202")
+					(reference "C202")
 					(unit 1)
 				)
@@
 		(in_pos_files yes)
 		(dnp no)
-		(property "Reference" "C1205"
+		(property "Reference" "C205"
 			(at 198.12 96.52 0)
 			(show_name no)
@@
 		)
 		(property "LCSC" ""
-			(at 195.58 97.79 0)
-			(hide yes)
-			(show_name no)
-			(do_not_autoplace no)
-			(effects
-				(font
-					(size 1.27 1.27)
-				)
-			)
-		)
-		(property "Sim.Enable" ""
 			(at 195.58 97.79 0)
 			(hide yes)
@@
 			(project "plug"
 				(path "/6c8448b4-b04d-47e1-934e-e40cbe27a7be/095cddf1-6522-4d3b-885d-b21acd91d0c6"
-					(reference "C1205")
+					(reference "C205")
 					(unit 1)
 				)
@@
 		(in_pos_files yes)
 		(dnp no)
-		(property "Reference" "#PWR01206"
+		(property "Reference" "#PWR0206"
 			(at 185.42 106.68 0)
 			(hide yes)
@@
 			(project "plug"
 				(path "/6c8448b4-b04d-47e1-934e-e40cbe27a7be/095cddf1-6522-4d3b-885d-b21acd91d0c6"
-					(reference "#PWR01206")
+					(reference "#PWR0206")
 					(unit 1)
 				)
@@
 		(in_pos_files yes)
 		(dnp no)
-		(property "Reference" "#PWR01207"
+		(property "Reference" "#PWR0207"
 			(at 195.58 106.68 0)
 			(hide yes)
@@
 			(project "plug"
 				(path "/6c8448b4-b04d-47e1-934e-e40cbe27a7be/095cddf1-6522-4d3b-885d-b21acd91d0c6"
-					(reference "#PWR01207")
+					(reference "#PWR0207")
 					(unit 1)
 				)
@@
 		(in_pos_files yes)
 		(dnp no)
-		(property "Reference" "#PWR01201"
+		(property "Reference" "#PWR0201"
 			(at 97.79 106.68 0)
 			(hide yes)
@@
 			(project "plug"
 				(path "/6c8448b4-b04d-47e1-934e-e40cbe27a7be/095cddf1-6522-4d3b-885d-b21acd91d0c6"
-					(reference "#PWR01201")
+					(reference "#PWR0201")
 					(unit 1)
 				)
@@
 		(in_pos_files yes)
 		(dnp no)
-		(property "Reference" "#PWR01202"
+		(property "Reference" "#PWR0202"
 			(at 109.22 106.68 0)
 			(hide yes)
@@
 			(project "plug"
 				(path "/6c8448b4-b04d-47e1-934e-e40cbe27a7be/095cddf1-6522-4d3b-885d-b21acd91d0c6"
-					(reference "#PWR01202")
+					(reference "#PWR0202")
 					(unit 1)
 				)
@@
 		(in_pos_files yes)
 		(dnp no)
-		(property "Reference" "C1203"
+		(property "Reference" "C203"
 			(at 122.682 109.22 90)
 			(show_name no)
@@
 		)
 		(property "LCSC" ""
-			(at 125.73 105.41 90)
-			(hide yes)
-			(show_name no)
-			(do_not_autoplace no)
-			(effects
-				(font
-					(size 1.27 1.27)
-				)
-			)
-		)
-		(property "Sim.Enable" ""
 			(at 125.73 105.41 90)
 			(hide yes)
@@
 			(project "plug"
 				(path "/6c8448b4-b04d-47e1-934e-e40cbe27a7be/095cddf1-6522-4d3b-885d-b21acd91d0c6"
-					(reference "C1203")
+					(reference "C203")
 					(unit 1)
 				)
@@
 		(in_pos_files yes)
 		(dnp no)
-		(property "Reference" "C1204"
+		(property "Reference" "C204"
 			(at 187.96 96.52 0)
 			(show_name no)
@@
 		)
 		(property "LCSC" ""
-			(at 185.42 97.79 0)
-			(hide yes)
-			(show_name no)
-			(do_not_autoplace no)
-			(effects
-				(font
-					(size 1.27 1.27)
-				)
-			)
-		)
-		(property "Sim.Enable" ""
 			(at 185.42 97.79 0)
 			(hide yes)
@@
 			(project "plug"
 				(path "/6c8448b4-b04d-47e1-934e-e40cbe27a7be/095cddf1-6522-4d3b-885d-b21acd91d0c6"
-					(reference "C1204")
+					(reference "C204")
 					(unit 1)
 				)
@@
 		(in_pos_files yes)
 		(dnp no)
-		(property "Reference" "#PWR01203"
+		(property "Reference" "#PWR0203"
 			(at 116.84 105.41 0)
 			(hide yes)
@@
 			(project "plug"
 				(path "/6c8448b4-b04d-47e1-934e-e40cbe27a7be/095cddf1-6522-4d3b-885d-b21acd91d0c6"
-					(reference "#PWR01203")
+					(reference "#PWR0203")
 					(unit 1)
 				)
@@
 		(in_pos_files yes)
 		(dnp no)
-		(property "Reference" "#PWR01204"
+		(property "Reference" "#PWR0204"
 			(at 129.54 110.49 0)
 			(hide yes)
@@
 			(project "plug"
 				(path "/6c8448b4-b04d-47e1-934e-e40cbe27a7be/095cddf1-6522-4d3b-885d-b21acd91d0c6"
-					(reference "#PWR01204")
+					(reference "#PWR0204")
 					(unit 1)
 				)
@@
 		(in_pos_files yes)
 		(dnp no)
-		(property "Reference" "#PWR01205"
+		(property "Reference" "#PWR0205"
 			(at 148.59 121.92 0)
 			(hide yes)
@@
 			(project "plug"
 				(path "/6c8448b4-b04d-47e1-934e-e40cbe27a7be/095cddf1-6522-4d3b-885d-b21acd91d0c6"
-					(reference "#PWR01205")
+					(reference "#PWR0205")
 					(unit 1)
 				)
@@
 		(in_pos_files yes)
 		(dnp no)
-		(property "Reference" "C1201"
+		(property "Reference" "C201"
 			(at 100.33 96.52 0)
 			(show_name no)
@@
 		)
 		(property "LCSC" ""
-			(at 97.79 97.79 0)
-			(hide yes)
-			(show_name no)
-			(do_not_autoplace no)
-			(effects
-				(font
-					(size 1.27 1.27)
-				)
-			)
-		)
-		(property "Sim.Enable" ""
 			(at 97.79 97.79 0)
 			(hide yes)
@@
 			(project "plug"
 				(path "/6c8448b4-b04d-47e1-934e-e40cbe27a7be/095cddf1-6522-4d3b-885d-b21acd91d0c6"
-					(reference "C1201")
+					(reference "C201")
 					(unit 1)
 				)
