File: hardware/plug/plug.kicad_pcb (KiCad board)
At the start: 4 copper layers, 50 x 34.5 mm, 56 parts, among them J101 Cortex, J102 DX07S016JA3, J1101 NE8FAH, J201 SJ2-25404B-SMT-TR, J301 SJ2-25404B-SMT-TR, SW101 SKSG, U101 ATSAMD51J, U102 TPS78433QWDRBRQ1, U1101 THVD2442, U1201 TPSM33620S5QRDNRQ1, U201 TLP2361, U301 74AHC1G125, Y101 32k768

Commit message: Good Bye Imperial
Parts:
- C101, C102, C103, C104, C105, C106, C107, C108, C109, C1101, C1202, C1203, C201, C202, C301: footprint V2_Capacitor_SMD:C_0603 -> V2_Capacitor_SMD:C_1608
- C110, C111: footprint V2_Capacitor_SMD:C_0805 -> V2_Capacitor_SMD:C_2012
- C1201, C1204, C1205: footprint V2_Capacitor_SMD:C_1210 -> V2_Capacitor_SMD:C_3225
- D103: footprint V2_LED:LED_0603 -> V2_LED:LED_1608
- R101, R102, R103, R104, R1101, R201, R301, R302: footprint V2_Resistor_SMD:R_0603 -> V2_Resistor_SMD:R_1608
- TVS301: footprint V2_Diode_SMD:D_0603 -> V2_Diode_SMD:D_1608

Commit message: Refresh
Parts:
- renumbered C1201 to C201, C1202 to C202, C1203 to C203, C1204 to C204, C1205 to C205, C1101 to C301, C201 to C401, C202 to C402, C301 to C501, D201 to D401, D301 to D501, J1101 to J301, J201 to J401, J301 to J501, R1101 to R301, R201 to R401, R301 to R501, R302 to R502, TVS301 to TVS501, U1201 to U201, U1101 to U301, U201 to U401, U301 to U501

Commit message: Refresh
Parts:
- INFO102: value Layer_Numbers -> Layer_Numbers-4; footprint V2_Production:Layer_Numbers -> V2_Production:Layer_Numbers-4
