File: hardware/socket/MIDIOut.kicad_sch (KiCad schematic)
At the start: 7 parts, among them J401 SJ2-25404B-SMT-TR, U401 74AHC1G125

Commit message: Good Bye Imperial
Parts:
- C401: footprint V2_Capacitor_SMD:C_0603 -> V2_Capacitor_SMD:C_1608; symbol V2_Capacitor:0603_0u1 -> V2_Capacitor:1608_0u1
- R401, R402: footprint V2_Resistor_SMD:R_0603 -> V2_Resistor_SMD:R_1608; symbol V2_Resistor:0603_220R -> V2_Resistor:1608_220R
- TVS401: footprint V2_Diode_SMD:D_0603 -> V2_Diode_SMD:D_1608
Changed lines of the file:
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@@
 	(title_block
 		(title "V2 connect-socket")
-		(date "2026-04-23")
+		(date "2026-05-11")
 		(rev "2026-04-23")
 		(company "Versio Duo")
@@
 	)
 	(symbol
-		(lib_id "V2_Capacitor:0603_0u1")
+		(lib_id "V2_Capacitor:1608_0u1")
 		(at 106.68 86.36 0)
 		(unit 1)
@@
 			)
 		)
-		(property "Footprint" "V2_Capacitor_SMD:C_0603"
+		(property "Footprint" "V2_Capacitor_SMD:C_1608"
 			(at 106.68 103.378 0)
 			(hide yes)
@@
 	)
 	(symbol
-		(lib_id "V2_Resistor:0603_220R")
+		(lib_id "V2_Resistor:1608_220R")
 		(at 142.24 109.22 90)
 		(unit 1)
@@
 			)
 		)
-		(property "Footprint" "V2_Resistor_SMD:R_0603"
+		(property "Footprint" "V2_Resistor_SMD:R_1608"
 			(at 157.988 109.22 0)
 			(hide yes)
@@
 	)
 	(symbol
-		(lib_id "V2_Resistor:0603_220R")
+		(lib_id "V2_Resistor:1608_220R")
 		(at 156.21 87.63 180)
 		(unit 1)
@@
 			)
 		)
-		(property "Footprint" "V2_Resistor_SMD:R_0603"
+		(property "Footprint" "V2_Resistor_SMD:R_1608"
 			(at 156.21 71.882 0)
 			(hide yes)
@@
 			)
 		)
-		(property "Footprint" "V2_Diode_SMD:D_0603"
+		(property "Footprint" "V2_Diode_SMD:D_1608"
 			(at 121.285 113.03 0)
 			(hide yes)
