File: hardware/socket/PowerSupply.kicad_sch (KiCad schematic)
At the start: 6 parts, among them U601 TPSM33620S5QRDNRQ1

Commit message: Split into socket and plug
Other:
- title: V2 connect -> V2 connect-socket
Changed lines of the file:
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@@
 	(paper "A4")
 	(title_block
-		(title "V2 connect")
-		(date "2026-04-14")
-		(rev "2026-04-14")
+		(title "V2 connect-socket")
+		(date "2026-04-23")
+		(rev "2026-04-23")
 		(company "Versio Duo")
 		(comment 1 "V2 Link Connector")
@@
 		)
 		(instances
-			(project "connect"
+			(project "socket"
 				(path "/6c8448b4-b04d-47e1-934e-e40cbe27a7be/095cddf1-6522-4d3b-885d-b21acd91d0c6"
 					(reference "U601")
@@
 		)
 		(instances
-			(project "connect"
+			(project "socket"
 				(path "/6c8448b4-b04d-47e1-934e-e40cbe27a7be/095cddf1-6522-4d3b-885d-b21acd91d0c6"
 					(reference "C602")
@@
 		)
 		(instances
-			(project "connect"
+			(project "socket"
 				(path "/6c8448b4-b04d-47e1-934e-e40cbe27a7be/095cddf1-6522-4d3b-885d-b21acd91d0c6"
 					(reference "C605")
@@
 		(in_pos_files yes)
 		(dnp no)
-		(property "Reference" "#PWR606"
+		(property "Reference" "#PWR0606"
 			(at 185.42 106.68 0)
 			(hide yes)
@@
 		)
 		(instances
-			(project "connect"
+			(project "socket"
 				(path "/6c8448b4-b04d-47e1-934e-e40cbe27a7be/095cddf1-6522-4d3b-885d-b21acd91d0c6"
-					(reference "#PWR606")
+					(reference "#PWR0606")
 					(unit 1)
 				)
@@
 		(in_pos_files yes)
 		(dnp no)
-		(property "Reference" "#PWR607"
+		(property "Reference" "#PWR0607"
 			(at 195.58 106.68 0)
 			(hide yes)
@@
 		)
 		(instances
-			(project "connect"
+			(project "socket"
 				(path "/6c8448b4-b04d-47e1-934e-e40cbe27a7be/095cddf1-6522-4d3b-885d-b21acd91d0c6"
-					(reference "#PWR607")
+					(reference "#PWR0607")
 					(unit 1)
 				)
@@
 		(in_pos_files yes)
 		(dnp no)
-		(property "Reference" "#PWR601"
+		(property "Reference" "#PWR0601"
 			(at 97.79 106.68 0)
 			(hide yes)
@@
 		)
 		(instances
-			(project "connect"
+			(project "socket"
 				(path "/6c8448b4-b04d-47e1-934e-e40cbe27a7be/095cddf1-6522-4d3b-885d-b21acd91d0c6"
-					(reference "#PWR601")
+					(reference "#PWR0601")
 					(unit 1)
 				)
@@
 		(in_pos_files yes)
 		(dnp no)
-		(property "Reference" "#PWR602"
+		(property "Reference" "#PWR0602"
 			(at 109.22 106.68 0)
 			(hide yes)
@@
 		)
 		(instances
-			(project "connect"
+			(project "socket"
 				(path "/6c8448b4-b04d-47e1-934e-e40cbe27a7be/095cddf1-6522-4d3b-885d-b21acd91d0c6"
-					(reference "#PWR602")
+					(reference "#PWR0602")
 					(unit 1)
 				)
@@
 		)
 		(instances
-			(project "connect"
+			(project "socket"
 				(path "/6c8448b4-b04d-47e1-934e-e40cbe27a7be/095cddf1-6522-4d3b-885d-b21acd91d0c6"
 					(reference "C603")
@@
 		)
 		(instances
-			(project "connect"
+			(project "socket"
 				(path "/6c8448b4-b04d-47e1-934e-e40cbe27a7be/095cddf1-6522-4d3b-885d-b21acd91d0c6"
 					(reference "C604")
@@
 		(in_pos_files yes)
 		(dnp no)
-		(property "Reference" "#PWR603"
+		(property "Reference" "#PWR0603"
 			(at 116.84 105.41 0)
 			(hide yes)
@@
 		)
 		(instances
-			(project "connect"
+			(project "socket"
 				(path "/6c8448b4-b04d-47e1-934e-e40cbe27a7be/095cddf1-6522-4d3b-885d-b21acd91d0c6"
-					(reference "#PWR603")
+					(reference "#PWR0603")
 					(unit 1)
 				)
@@
 		(in_pos_files yes)
 		(dnp no)
-		(property "Reference" "#PWR604"
+		(property "Reference" "#PWR0604"
 			(at 129.54 110.49 0)
 			(hide yes)
@@
 		)
 		(instances
-			(project "connect"
+			(project "socket"
 				(path "/6c8448b4-b04d-47e1-934e-e40cbe27a7be/095cddf1-6522-4d3b-885d-b21acd91d0c6"
-					(reference "#PWR604")
+					(reference "#PWR0604")
 					(unit 1)
 				)
@@
 		(in_pos_files yes)
 		(dnp no)
-		(property "Reference" "#PWR605"
+		(property "Reference" "#PWR0605"
 			(at 148.59 121.92 0)
 			(hide yes)
@@
 		)
 		(instances
-			(project "connect"
+			(project "socket"
 				(path "/6c8448b4-b04d-47e1-934e-e40cbe27a7be/095cddf1-6522-4d3b-885d-b21acd91d0c6"
-					(reference "#PWR605")
+					(reference "#PWR0605")
 					(unit 1)
 				)
@@
 		)
 		(instances
-			(project "connect"
+			(project "socket"
 				(path "/6c8448b4-b04d-47e1-934e-e40cbe27a7be/095cddf1-6522-4d3b-885d-b21acd91d0c6"
 					(reference "C601")

Commit message: Good Bye Imperial
Parts:
- C601: footprint V2_Capacitor_SMD:C_1210 -> V2_Capacitor_SMD:C_3225; symbol V2_Capacitor:1210_10u -> V2_Capacitor:3225_10u
- C602: footprint V2_Capacitor_SMD:C_0603 -> V2_Capacitor_SMD:C_1608; symbol V2_Capacitor:0603_0u1 -> V2_Capacitor:1608_0u1
- C603: footprint V2_Capacitor_SMD:C_0603 -> V2_Capacitor_SMD:C_1608; symbol V2_Capacitor:0603_1u -> V2_Capacitor:1608_1u
- C604, C605: footprint V2_Capacitor_SMD:C_1210 -> V2_Capacitor_SMD:C_3225; symbol V2_Capacitor:1210_22u -> V2_Capacitor:3225_22u
Changed lines of the file:
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@@
 	(title_block
 		(title "V2 connect-socket")
-		(date "2026-04-23")
+		(date "2026-05-11")
 		(rev "2026-04-23")
 		(company "Versio Duo")
@@
 	)
 	(symbol
-		(lib_id "V2_Capacitor:0603_0u1")
+		(lib_id "V2_Capacitor:1608_0u1")
 		(at 109.22 97.79 0)
 		(unit 1)
@@
 			)
 		)
-		(property "Footprint" "V2_Capacitor_SMD:C_0603"
+		(property "Footprint" "V2_Capacitor_SMD:C_1608"
 			(at 109.22 114.808 0)
 			(hide yes)
@@
 	)
 	(symbol
-		(lib_id "V2_Capacitor:1210_22u")
+		(lib_id "V2_Capacitor:3225_22u")
 		(at 195.58 97.79 0)
 		(unit 1)
@@
 			)
 		)
-		(property "Footprint" "V2_Capacitor_SMD:C_1210"
+		(property "Footprint" "V2_Capacitor_SMD:C_3225"
 			(at 195.58 114.808 0)
 			(hide yes)
@@
 	)
 	(symbol
-		(lib_id "V2_Capacitor:0603_1u")
+		(lib_id "V2_Capacitor:1608_1u")
 		(at 125.73 105.41 90)
 		(unit 1)
@@
 			)
 		)
-		(property "Footprint" "V2_Capacitor_SMD:C_0603"
+		(property "Footprint" "V2_Capacitor_SMD:C_1608"
 			(at 142.748 105.41 0)
 			(hide yes)
@@
 	)
 	(symbol
-		(lib_id "V2_Capacitor:1210_22u")
+		(lib_id "V2_Capacitor:3225_22u")
 		(at 185.42 97.79 0)
 		(unit 1)
@@
 			)
 		)
-		(property "Footprint" "V2_Capacitor_SMD:C_1210"
+		(property "Footprint" "V2_Capacitor_SMD:C_3225"
 			(at 185.42 114.808 0)
 			(hide yes)
@@
 	)
 	(symbol
-		(lib_id "V2_Capacitor:1210_10u")
+		(lib_id "V2_Capacitor:3225_10u")
 		(at 97.79 97.79 0)
 		(unit 1)
@@
 			)
 		)
-		(property "Footprint" "V2_Capacitor_SMD:C_1210"
+		(property "Footprint" "V2_Capacitor_SMD:C_3225"
 			(at 97.79 114.808 0)
 			(hide yes)
