File: hardware/socket/socket.kicad_pcb (KiCad board)
At the start: 4 copper layers, 80 x 34.5 mm, 80 parts, among them J101 Cortex, J102 DX07S016JA3, J201 NE8FAH, J301 SJ2-25404B-SMT-TR, J401 SJ2-25404B-SMT-TR, SW101 SKSG, SW102 SKSG, SW103 SKSG, SW104 SKSG, SW105 SKSG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

Commit message: Good Bye Imperial
Parts:
- C101, C102, C103, C104, C105, C106, C107, C108, C110, C201, C301, C302, C401, C602, C603: footprint V2_Capacitor_SMD:C_0603 -> V2_Capacitor_SMD:C_1608
- C109, C111: footprint V2_Capacitor_SMD:C_0805 -> V2_Capacitor_SMD:C_2012
- C601, C604, C605: footprint V2_Capacitor_SMD:C_1210 -> V2_Capacitor_SMD:C_3225
- D101: footprint V2_LED:LED_0603 -> V2_LED:LED_1608
- R101, R102, R103, R104, R201, R301, R401, R402: footprint V2_Resistor_SMD:R_0603 -> V2_Resistor_SMD:R_1608
- TVS401: footprint V2_Diode_SMD:D_0603 -> V2_Diode_SMD:D_1608
Changed lines of the file:
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@@
 	(paper "A4")
 	(title_block
-		(date "2026-04-23")
+		(date "2026-05-11")
 		(rev "2026-04-23")
 	)
@@
 		)
 	)
-	(footprint "V2_Capacitor_SMD:C_0603"
+	(footprint "V2_Capacitor_SMD:C_1608"
 		(layer "F.Cu")
 		(at 69.5 102.75)
@@
 			)
 		)
-		(property "Id" "Capacitor:0603_1u"
+		(property "Id" "Capacitor:1608_1u"
 			(at 0 0 0)
 			(unlocked yes)
@@
 		)
 	)
-	(footprint "V2_Capacitor_SMD:C_0603"
+	(footprint "V2_Capacitor_SMD:C_1608"
 		(layer "F.Cu")
 		(at 98.25 99)
@@
 			)
 		)
-		(property "Id" "Capacitor:0603_18p"
+		(property "Id" "Capacitor:1608_18p"
 			(at 0 0 0)
 			(unlocked yes)
@@
 		)
 	)
-	(footprint "V2_Capacitor_SMD:C_0603"
+	(footprint "V2_Capacitor_SMD:C_1608"
 		(layer "F.Cu")
 		(at 137 98 180)
@@
 			)
 		)
-		(property "Id" "Capacitor:0603_0u1"
+		(property "Id" "Capacitor:1608_0u1"
 			(at 0 0 180)
 			(unlocked yes)
@@
 		)
 	)
-	(footprint "V2_Resistor_SMD:R_0603"
+	(footprint "V2_Resistor_SMD:R_1608"
 		(layer "F.Cu")
 		(at 133.5 96.25 180)
@@
 			)
 		)
-		(property "Id" "Resistor:0603_5k1"
+		(property "Id" "Resistor:1608_5k1"
 			(at 0 0 180)
 			(unlocked yes)
@@
 		)
 	)
-	(footprint "V2_Capacitor_SMD:C_0603"
+	(footprint "V2_Capacitor_SMD:C_1608"
 		(layer "F.Cu")
 		(at 82.5 98 90)
@@
 			)
 		)
-		(property "Id" "Capacitor:0603_0u1"
+		(property "Id" "Capacitor:1608_0u1"
 			(at 0 0 90)
 			(unlocked yes)
@@
 		)
 	)
-	(footprint "V2_Capacitor_SMD:C_0603"
+	(footprint "V2_Capacitor_SMD:C_1608"
 		(layer "F.Cu")
 		(at 76.5 110.25 -90)
@@
 			)
 		)
-		(property "Id" "Capacitor:0603_0u1"
+		(property "Id" "Capacitor:1608_0u1"
 			(at 0 0 270)
 			(unlocked yes)
@@
 		)
 	)
-	(footprint "V2_Capacitor_SMD:C_0603"
+	(footprint "V2_Capacitor_SMD:C_1608"
 		(layer "F.Cu")
 		(at 90.75 87.75 180)
@@
 			)
 		)
-		(property "Id" "Capacitor:0603_0u1"
+		(property "Id" "Capacitor:1608_0u1"
 			(at 0 0 180)
 			(unlocked yes)
@@
 		)
 	)
-	(footprint "V2_Capacitor_SMD:C_0603"
+	(footprint "V2_Capacitor_SMD:C_1608"
 		(layer "F.Cu")
 		(at 98.25 96.5)
@@
 			)
 		)
-		(property "Id" "Capacitor:0603_18p"
+		(property "Id" "Capacitor:1608_18p"
 			(at 0 0 0)
 			(unlocked yes)
@@
 		)
 	)
-	(footprint "V2_Capacitor_SMD:C_1210"
+	(footprint "V2_Capacitor_SMD:C_3225"
 		(layer "F.Cu")
 		(at 70.75 94.5)
@@
 			)
 		)
-		(property "Id" "Capacitor:1210_10u"
+		(property "Id" "Capacitor:3225_10u"
 			(at 0 0 0)
 			(unlocked yes)
@@
 		)
 	)
-	(footprint "V2_Resistor_SMD:R_0603"
+	(footprint "V2_Resistor_SMD:R_1608"
 		(layer "F.Cu")
 		(at 116 114.5 180)
@@
 			)
 		)
-		(property "Id" "Resistor:0603_220R"
+		(property "Id" "Resistor:1608_220R"
 			(at 0 0 180)
 			(unlocked yes)
@@
 		)
 	)
-	(footprint "V2_Capacitor_SMD:C_0603"
+	(footprint "V2_Capacitor_SMD:C_1608"
 		(layer "F.Cu")
 		(at 86.25 101.75 -90)
@@
 			)
 		)
-		(property "Id" "Capacitor:0603_10u"
+		(property "Id" "Capacitor:1608_10u"
 			(at 0 0 270)
 			(unlocked yes)
@@
 		)
 	)
-	(footprint "V2_Resistor_SMD:R_0603"
+	(footprint "V2_Resistor_SMD:R_1608"
 		(layer "F.Cu")
 		(at 133.5 87.25 180)
@@
 			)
 		)
-		(property "Id" "Resistor:0603_5k1"
+		(property "Id" "Resistor:1608_5k1"
 			(at 0 0 180)
 			(unlocked yes)
@@
 		)
 	)
-	(footprint "V2_Capacitor_SMD:C_0603"
+	(footprint "V2_Capacitor_SMD:C_1608"
 		(layer "F.Cu")
 		(at 105 114.5 180)
@@
 			)
 		)
-		(property "Id" "Capacitor:0603_0u1"
+		(property "Id" "Capacitor:1608_0u1"
 			(at 0 0 180)
 			(unlocked yes)
@@
 		)
 	)
-	(footprint "V2_Capacitor_SMD:C_0805"
+	(footprint "V2_Capacitor_SMD:C_2012"
 		(layer "F.Cu")
 		(at 103.25 87.5 -90)
@@
 			)
 		)
-		(property "Id" "Capacitor:0805_10u"
+		(property "Id" "Capacitor:2012_10u"
 			(at 0 0 270)
 			(unlocked yes)
@@
 		)
 	)
-	(footprint "V2_Capacitor_SMD:C_0603"
+	(footprint "V2_Capacitor_SMD:C_1608"
 		(layer "F.Cu")
 		(at 77 88.5)
@@
 			)
 		)
-		(property "Id" "Capacitor:0603_0u1"
+		(property "Id" "Capacitor:1608_0u1"
 			(at 0 0 0)
 			(unlocked yes)
@@
 		)
 	)
-	(footprint "V2_Resistor_SMD:R_0603"
+	(footprint "V2_Resistor_SMD:R_1608"
 		(layer "F.Cu")
 		(at 78.75 107.25)
@@
 			)
 		)
-		(property "Id" "Resistor:0603_100R"
+		(property "Id" "Resistor:1608_100R"
 			(at 0 0 0)
 			(unlocked yes)
@@
 		(embedded_fonts no)
 	)
-	(footprint "V2_Resistor_SMD:R_0603"
+	(footprint "V2_Resistor_SMD:R_1608"
 		(layer "F.Cu")
 		(at 125.25 111.5 180)
@@
 			)
 		)
-		(property "Id" "Resistor:0603_220R"
+		(property "Id" "Resistor:1608_220R"
 			(at 0 0 180)
 			(unlocked yes)
@@
 		)
 	)
-	(footprint "V2_Resistor_SMD:R_0603"
+	(footprint "V2_Resistor_SMD:R_1608"
 		(layer "F.Cu")
 		(at 125.25 113.25)
@@
 			)
 		)
-		(property "Id" "Resistor:0603_220R"
+		(property "Id" "Resistor:1608_220R"
 			(at 0 0 0)
 			(unlocked yes)
@@
 		)
 	)
-	(footprint "V2_Resistor_SMD:R_0603"
+	(footprint "V2_Resistor_SMD:R_1608"
 		(layer "F.Cu")
 		(at 87.25 111.75 90)
@@
 			)
 		)
-		(property "Id" "Resistor:0603_330R"
+		(property "Id" "Resistor:1608_330R"
 			(at 0 0 90)
 			(unlocked yes)
@@
 		)
 	)
-	(footprint "V2_Capacitor_SMD:C_1210"
+	(footprint "V2_Capacitor_SMD:C_3225"
 		(layer "F.Cu")
 		(at 66 92.75 180)
@@
 			)
 		)
-		(property "Id" "Capacitor:1210_22u"
+		(property "Id" "Capacitor:3225_22u"
 			(at 0 0 180)
 			(unlocked yes)
@@
 		)
 	)
-	(footprint "V2_LED:LED_0603"
+	(footprint "V2_LED:LED_1608"
 		(layer "F.Cu")
 		(at 85.75 111.75 90)
@@
 			)
 		)
-		(property "Sim.Pins" "1=K 2=A"
+		(property "Mouser" "755-SML-D12D1WT86"
 			(at 0 0 90)
 			(unlocked yes)
@@
 			)
 		)
-		(property "Mouser" "755-SML-D12D1WT86"
+		(property "Product" "SML-D12D1WT86"
 			(at 0 0 90)
 			(unlocked yes)
@@
 			)
 		)
-		(property "Product" "SML-D12D1WT86"
+		(property "Manufacturer" "ROHM Semiconductor "
 			(at 0 0 90)
 			(unlocked yes)
@@
 			)
 		)
-		(property "Manufacturer" "ROHM Semiconductor "
+		(property "Id" "LED:1608_Orange"
 			(at 0 0 90)
 			(unlocked yes)
@@
 			)
 		)
-		(property "Id" "LED:0603_Orange"
+		(property "Rating" "605nm"
 			(at 0 0 90)
 			(unlocked yes)
@@
 			)
 		)
-		(property "Rating" "605nm"
+		(property "Sim.Pins" "1=K 2=A"
 			(at 0 0 90)
 			(unlocked yes)
@@
 		)
 	)
-	(footprint "V2_Capacitor_SMD:C_0603"
+	(footprint "V2_Capacitor_SMD:C_1608"
 		(layer "F.Cu")
 		(at 82.75 90.25 90)
@@
 			)
 		)
-		(property "Id" "Capacitor:0603_0u1"
+		(property "Id" "Capacitor:1608_0u1"
 			(at 0 0 90)
 			(unlocked yes)
@@
 		)
 	)
-	(footprint "V2_Capacitor_SMD:C_0603"
+	(footprint "V2_Capacitor_SMD:C_1608"
 		(layer "F.Cu")
 		(at 95.25 94 -90)
@@
 			)
 		)
-		(property "Id" "Capacitor:0603_0u1"
+		(property "Id" "Capacitor:1608_0u1"
 			(at 0 0 270)
 			(unlocked yes)
@@
 		)
 	)
-	(footprint "V2_Capacitor_SMD:C_0805"
+	(footprint "V2_Capacitor_SMD:C_2012"
 		(layer "F.Cu")
 		(at 109.75 87.5 -90)
@@
 			)
 		)
-		(property "Id" "Capacitor:0805_10u"
+		(property "Id" "Capacitor:2012_10u"
 			(at 0 0 270)
 			(unlocked yes)
@@
 		)
 	)
-	(footprint "V2_Capacitor_SMD:C_1210"
+	(footprint "V2_Capacitor_SMD:C_3225"
 		(layer "F.Cu")
 		(at 66 96 180)
@@
 			)
 		)
-		(property "Id" "Capacitor:1210_22u"
+		(property "Id" "Capacitor:3225_22u"
 			(at 0 0 180)
 			(unlocked yes)
@@
 		)
 	)
-	(footprint "V2_Capacitor_SMD:C_0603"
+	(footprint "V2_Capacitor_SMD:C_1608"
 		(layer "F.Cu")
 		(at 70 97)
@@
 			)
 		)
-		(property "Id" "Capacitor:0603_0u1"
+		(property "Id" "Capacitor:1608_0u1"
 			(at 0 0 0)
 			(unlocked yes)
@@
 		)
 	)
-	(footprint "V2_Capacitor_SMD:C_0603"
+	(footprint "V2_Capacitor_SMD:C_1608"
 		(layer "F.Cu")
 		(at 88.5 101.75 -90)
@@
 			)
 		)
-		(property "Id" "Capacitor:0603_0u1"
+		(property "Id" "Capacitor:1608_0u1"
 			(at 0 0 270)
 			(unlocked yes)
@@
 		(embedded_fonts no)
 	)
-	(footprint "V2_Diode_SMD:D_0603"
+	(footprint "V2_Diode_SMD:D_1608"
 		(layer "F.Cu")
 		(at 125.25 114.75 180)
@@
 		)
 	)
-	(footprint "V2_Capacitor_SMD:C_0603"
+	(footprint "V2_Capacitor_SMD:C_1608"
 		(layer "F.Cu")
 		(at 121.5 111.5 180)
@@
 			)
 		)
-		(property "Id" "Capacitor:0603_0u1"
+		(property "Id" "Capacitor:1608_0u1"
 			(at 0 0 180)
 			(unlocked yes)
@@
 		)
 	)
-	(footprint "V2_Resistor_SMD:R_0603"
+	(footprint "V2_Resistor_SMD:R_1608"
 		(layer "F.Cu")
 		(at 90.25 112.25 90)
@@
 			)
 		)
-		(property "Id" "Resistor:0603_100k"
+		(property "Id" "Resistor:1608_100k"
 			(at 0 0 90)
 			(unlocked yes)

Commit message: Refresh
Parts:
- INFO102: value Layer_Numbers -> Layer_Numbers-4; footprint V2_Production:Layer_Numbers -> V2_Production:Layer_Numbers-4
- moved INFO102 9.25 mm to (65.8, 116.5)
Routing:
- net /USB+: track 71.5 -> 70.3 mm
- net /USB-: track 73.4 -> 72.9 mm
